File: pcb/base-1.0/poe.sch (KiCad schematic (older format))
At the start: 44 parts

Commit message: wip
Parts:
- added C314: 1uF, symbol Device:C
- added C317: 10pF, symbol Device:C
- added C318: 15nF, symbol Device:C
- added C319: 100pF, symbol Device:C
- added C320: 100uF, symbol Device:C
- added C321: 22uF, symbol Device:C
- added D308: BAV99, symbol Device:D_x2_Serial_ACK
- added D309, D311: BAS16, symbol Device:D
- added D310, D312: 12V, symbol Device:D_Zener
- added L303: 22uH, symbol Device:L_Core_Ferrite
- added Q303: Si7852DP, symbol Device:Q_NMOS_DGS
- added Q304, Q305: MMBTA06, symbol Device:Q_NPN_BCE
- added Q306: Si4850EY, symbol Device:Q_NMOS_DGS
- added R312: 2.49k, symbol Device:R
- added R314, R315: 10k, symbol Device:R
- added R316: 41.2k, symbol Device:R
- added R317: 11k, symbol Device:R
- added R318: 49.9, symbol Device:R
- added R319, R320: 2k, symbol Device:R
- added U303: TL431D, Package_SO:SOIC-8_3.9x4.9mm_P1.27mm, symbol Reference_Voltage:TL431D
- C307: renamed from C?; value 1uH -> 1uF
- C309: renamed from C?; value 22uH -> 22uF; Voltage (none) -> 25V
- L301: renamed from L?; mpn (none) -> 74404043102A
- gave numbers to parts that had none: 41
Connections:
- net labels added: Vout
- wire segments 183 -> 273

Commit message: wip
Parts:
- C?: renamed from C314; value 1uF -> C
- D301, D302: value D_Bridge_+-AA -> CDBHD1100L-G
- renumbered C318 to C?, C317 to C?, D308 to D?, R318 to R?, R317 to R?, R316 to R?, R315 to R?, U303 to U?
Connections:
- net GND: now also D304.1 (K)
- net at NT301.1, NT301.3, R301.2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: no longer D304.1 (K)
- net Vin_A1: now reaches D301.3 (~~)
- net Vin_A2: now reaches D301.4 (~~)
- net Vin_B1: now reaches D302.3 (~~)
- net Vin_B2: now reaches D302.4 (~~)
Other:
- moved on the sheet: C301, C302, C304, C306, C307, C309, C310, C313, C315, C?, D301, D302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

Commit message: wip
Parts:
- gave numbers to parts that had none: 9
Changed lines of the file:
@@
 	10000 9300 10100 9300
 $Comp
-L Device:C C?
+L Device:C C317
 U 1 1 5D28C6A9
 P 9850 9300
-F 0 "C?" V 9598 9300 50  0000 C CNN
+F 0 "C317" V 9598 9300 50  0000 C CNN
 F 1 "10pF" V 9689 9300 50  0000 C CNN
 F 2 "" H 9888 9150 50  0001 C CNN
@@
 	8800 9700 9200 9700
 $Comp
-L Device:C C?
+L Device:C C318
 U 1 1 5D24F557
 P 9850 9700
-F 0 "C?" V 9598 9700 50  0000 C CNN
+F 0 "C318" V 9598 9700 50  0000 C CNN
 F 1 "15nF" V 9689 9700 50  0000 C CNN
 F 2 "" H 9888 9550 50  0001 C CNN
@@
 $EndComp
 $Comp
-L Device:R R?
+L Device:R R315
 U 1 1 5D24EE83
 P 9450 9700
-F 0 "R?" V 9657 9700 50  0000 C CNN
+F 0 "R315" V 9657 9700 50  0000 C CNN
 F 1 "10k" V 9566 9700 50  0000 C CNN
 F 2 "" V 9380 9700 50  0001 C CNN
@@
 	10500 9600 10500 9700
 $Comp
-L Device:R R?
+L Device:R R316
 U 1 1 5D1E0D58
 P 10500 9450
-F 0 "R?" H 10430 9404 50  0000 R CNN
+F 0 "R316" H 10430 9404 50  0000 R CNN
 F 1 "41.2k" H 10430 9495 50  0000 R CNN
 F 2 "" V 10430 9450 50  0001 C CNN
@@
 	10500 10500 10500 10400
 $Comp
-L Device:R R?
+L Device:R R317
 U 1 1 5D197E47
 P 10500 10150
-F 0 "R?" H 10430 10104 50  0000 R CNN
+F 0 "R317" H 10430 10104 50  0000 R CNN
 F 1 "11k" H 10430 10195 50  0000 R CNN
 F 2 "" V 10430 10150 50  0001 C CNN
@@
 $EndComp
 $Comp
-L power:GND #PWR?
+L power:GND #PWR0302
 U 1 1 5D194EBD
 P 10500 10500
-F 0 "#PWR?" H 10500 10250 50  0001 C CNN
+F 0 "#PWR0302" H 10500 10250 50  0001 C CNN
 F 1 "GND" H 10505 10327 50  0000 C CNN
 F 2 "" H 10500 10500 50  0001 C CNN
@@
 Connection ~ 8800 8800
 $Comp
-L Device:D_x2_Serial_ACK D?
+L Device:D_x2_Serial_ACK D308
 U 1 1 5D0EEC09
 P 8800 9300
-F 0 "D?" V 8846 9379 50  0000 L CNN
+F 0 "D308" V 8846 9379 50  0000 L CNN
 F 1 "BAV99" V 8755 9379 50  0000 L CNN
 F 2 "" H 8800 9300 50  0001 C CNN
@@
 $EndComp
 $Comp
-L Device:R R?
+L Device:R R318
 U 1 1 5D0EBF76
 P 10850 8800
-F 0 "R?" V 10643 8800 50  0000 C CNN
+F 0 "R318" V 10643 8800 50  0000 C CNN
 F 1 "49.9" V 10734 8800 50  0000 C CNN
 F 2 "" V 10780 8800 50  0001 C CNN
@@
 $EndComp
 $Comp
-L Reference_Voltage:TL431D U?
+L Reference_Voltage:TL431D U303
 U 1 1 5D0E968E
 P 8800 9900
-F 0 "U?" V 8846 9831 50  0000 R CNN
+F 0 "U303" V 8846 9831 50  0000 R CNN
 F 1 "TL431D" V 8755 9831 50  0000 R CNN
 F 2 "Package_SO:SOIC-8_3.9x4.9mm_P1.27mm" H 8800 9650 50  0001 C CIN
@@
 $EndComp
 $Comp
-L Device:C C?
+L Device:C C314
 U 1 1 5D1872D7
 P 8300 9950
-F 0 "C?" H 8415 9996 50  0000 L CNN
+F 0 "C314" H 8415 9996 50  0000 L CNN
 F 1 "C" H 8415 9905 50  0000 L CNN
 F 2 "" H 8338 9800 50  0001 C CNN
@@
 	9650 1600 9650 2500
 $Comp
-L unlockoslo:GND_ETH #PWR?
+L unlockoslo:GND_ETH #PWR0301
 U 1 1 5D7FEFF9
 P 3800 4200
-F 0 "#PWR?" H 3800 3950 50  0001 C CNN
+F 0 "#PWR0301" H 3800 3950 50  0001 C CNN
 F 1 "GND_ETH" H 3805 4027 50  0000 C CNN
 F 2 "" H 3800 4200 50  0001 C CNN

Commit message: wip
Parts:
- C301, C302, C303, C304, C305, C306, C307, C308, C309, C310, C311, C312, C313, C314, C315, C316, C317, C318, C319, C320, C321: footprint (none) -> Capacitor_SMD:C_0402_1005Metric
- D303, D304: footprint (none) -> Diode_SMD:D_SMA
- D305, D306, D307, D308, D309, D311: footprint (none) -> Diode_SMD:D_SOT-23_ANK
- FB301, FB302: footprint (none) -> Inductor_SMD:L_0603_1608Metric
- NT301: footprint (none) -> NetTie:NetTie-4_SMD_Pad0.5mm
- R301, R302, R303, R304, R305, R306, R307, R308, R309, R310, R311, R312, R313, R314, R315, R316, R317, R318, R319, R320: footprint (none) -> Resistor_SMD:R_0402_1005Metric

Commit message: wip
Parts:
- renumbered C306 to C305, C305 to C306, C309 to C308, C308 to C309, C313 to C312, C312 to C313
Changed lines of the file:
@@
 	9500 1800 9500 1900
 $Comp
-L unlockoslo:GND_ETH #PWR0129
+L unlockoslo:GND_ETH #PWR0123
 U 1 1 5D1429E9
 P 9500 1900
-F 0 "#PWR0129" H 9500 1650 50  0001 C CNN
+F 0 "#PWR0123" H 9500 1650 50  0001 C CNN
 F 1 "GND_ETH" H 9505 1727 50  0000 C CNN
 F 2 "" H 9500 1900 50  0001 C CNN
@@
 	10050 2500 10050 2600
 $Comp
-L unlockoslo:GND_ETH #PWR0130
+L unlockoslo:GND_ETH #PWR0124
 U 1 1 5D2A3598
 P 9550 2600
-F 0 "#PWR0130" H 9550 2350 50  0001 C CNN
+F 0 "#PWR0124" H 9550 2350 50  0001 C CNN
 F 1 "GND_ETH" H 9555 2427 50  0000 C CNN
 F 2 "" H 9550 2600 50  0001 C CNN
@@
 $EndComp
 $Comp
-L power:GND #PWR0131
+L power:GND #PWR0125
 U 1 1 5D2A4662
 P 10050 2600
-F 0 "#PWR0131" H 10050 2350 50  0001 C CNN
+F 0 "#PWR0125" H 10050 2350 50  0001 C CNN
 F 1 "GND" H 10055 2427 50  0000 C CNN
 F 2 "" H 10050 2600 50  0001 C CNN
@@
 	14000 1300 14200 1300
 $Comp
-L power:GND #PWR0132
+L power:GND #PWR0126
 U 1 1 5CD669FE
 P 14000 2900
-F 0 "#PWR0132" H 14000 2650 50  0001 C CNN
+F 0 "#PWR0126" H 14000 2650 50  0001 C CNN
 F 1 "GND" H 14005 2727 50  0000 C CNN
 F 2 "" H 14000 2900 50  0001 C CNN
@@
 	7200 1700 7200 1800
 $Comp
-L Device:C C308
+L Device:C C309
 U 1 1 5CD7E402
 P 6700 1550
-F 0 "C308" H 6815 1641 50  0000 L CNN
+F 0 "C309" H 6815 1641 50  0000 L CNN
 F 1 "22uF" H 6815 1550 50  0000 L CNN
 F 2 "Capacitor_SMD:C_0402_1005Metric" H 6738 1400 50  0001 C CNN
@@
 	7700 1400 7700 1300
 $Comp
-L Device:C C312
+L Device:C C313
 U 1 1 5CD71A0F
 P 7700 1550
-F 0 "C312" H 7815 1641 50  0000 L CNN
+F 0 "C313" H 7815 1641 50  0000 L CNN
 F 1 "1uF" H 7815 1550 50  0000 L CNN
 F 2 "Capacitor_SMD:C_0402_1005Metric" H 7738 1400 50  0001 C CNN
@@
 $EndComp
 $Comp
-L Device:C C305
+L Device:C C306
 U 1 1 5CD8D101
 P 6200 1550
-F 0 "C305" H 6315 1641 50  0000 L CNN
+F 0 "C306" H 6315 1641 50  0000 L CNN
 F 1 "1uF" H 6315 1550 50  0000 L CNN
 F 2 "Capacitor_SMD:C_0402_1005Metric" H 6238 1400 50  0001 C CNN
@@
 $EndComp
 Wire Wire Line
-	3800 3500 4400 3500
+	3800 3500 3900 3500
 Connection ~ 3800 3500
 Wire Wire Line
@@
 	1    0    0    -1
 $EndComp
-Text Label 4100 3500 0    50   ~ 0
+Text Label 4000 3500 0    50   ~ 0
 ETH_VSS
 Text Label 4100 1300 0    50   ~ 0
@@
 Connection ~ 7700 6600
 $Comp
-L Device:C C313
+L Device:C C312
 U 1 1 5CDDE6DB
 P 7450 6600
-F 0 "C313" V 7198 6600 50  0000 C CNN
+F 0 "C312" V 7198 6600 50  0000 C CNN
 F 1 "1uF" V 7289 6600 50  0000 C CNN
 F 2 "Capacitor_SMD:C_0402_1005Metric" H 7488 6450 50  0001 C CNN
@@
 	6800 5700 6800 5600
 $Comp
-L Device:C C306
+L Device:C C305
 U 1 1 5CE31A9B
 P 6100 5950
-F 0 "C306" H 5985 5904 50  0000 R CNN
+F 0 "C305" H 5985 5904 50  0000 R CNN
 F 1 "1uF" H 5985 5995 50  0000 R CNN
 F 2 "Capacitor_SMD:C_0402_1005Metric" H 6138 5800 50  0001 C CNN
@@
 	4600 7800 4600 7300
 $Comp
-L unlockoslo:GND_ETH #PWR0123
+L unlockoslo:GND_ETH #PWR0127
 U 1 1 5CEB780B
 P 4600 7900
-F 0 "#PWR0123" H 4600 7650 50  0001 C CNN
+F 0 "#PWR0127" H 4600 7650 50  0001 C CNN
 F 1 "GND_ETH" H 4605 7727 50  0000 C CNN
 F 2 "" H 4600 7900 50  0001 C CNN
@@
 Connection ~ 4600 7800
 $Comp
-L unlockoslo:GND_ETH #PWR0124
+L unlockoslo:GND_ETH #PWR0128
 U 1 1 5CEBD68D
 P 8500 7200
-F 0 "#PWR0124" H 8500 6950 50  0001 C CNN
+F 0 "#PWR0128" H 8500 6950 50  0001 C CNN
 F 1 "GND_ETH" H 8505 7027 50  0000 C CNN
 F 2 "" H 8500 7200 50  0001 C CNN
@@
 	6800 6200 6800 6100
 $Comp
-L unlockoslo:GND_ETH #PWR0125
+L unlockoslo:GND_ETH #PWR0129
 U 1 1 5CF3CBBF
 P 6800 6300
-F 0 "#PWR0125" H 6800 6050 50  0001 C CNN
+F 0 "#PWR0129" H 6800 6050 50  0001 C CNN
 F 1 "GND_ETH" H 6805 6127 50  0000 C CNN
 F 2 "" H 6800 6300 50  0001 C CNN
@@
 Connection ~ 7100 7500
 $Comp
-L Device:C C309
+L Device:C C308
 U 1 1 5D0400C8
 P 6600 7750
-F 0 "C309" H 6715 7841 50  0000 L CNN
+F 0 "C308" H 6715 7841 50  0000 L CNN
 F 1 "22uF" H 6715 7750 50  0000 L CNN
 F 2 "Capacitor_SMD:C_0402_1005Metric" H 6638 7600 50  0001 C CNN
@@
 	6600 8000 7100 8000
 $Comp
-L unlockoslo:GND_ETH #PWR0126
+L unlockoslo:GND_ETH #PWR0130
 U 1 1 5D056B5E
 P 7100 8100
-F 0 "#PWR0126" H 7100 7850 50  0001 C CNN
+F 0 "#PWR0130" H 7100 7850 50  0001 C CNN
 F 1 "GND_ETH" H 7105 7927 50  0000 C CNN
 F 2 "" H 7100 8100 50  0001 C CNN
@@
 	5700 8800 6100 8800
 $Comp
-L unlockoslo:GND_ETH #PWR0127
+L unlockoslo:GND_ETH #PWR0131
 U 1 1 5D0B93D2
 P 5700 9300
-F 0 "#PWR0127" H 5700 9050 50  0001 C CNN
+F 0 "#PWR0131" H 5700 9050 50  0001 C CNN
 F 1 "GND_ETH" H 5705 9127 50  0000 C CNN
 F 2 "" H 5700 9300 50  0001 C CNN
@@
 $EndComp
 $Comp
-L unlockoslo:GND_ETH #PWR0128
+L unlockoslo:GND_ETH #PWR0132
 U 1 1 5D10092F
 P 7100 9300
-F 0 "#PWR0128" H 7100 9050 50  0001 C CNN
+F 0 "#PWR0132" H 7100 9050 50  0001 C CNN
 F 1 "GND_ETH" H 7105 9127 50  0000 C CNN
 F 2 "" H 7100 9300 50  0001 C CNN
@@
 $EndComp
 $Comp
-L power:GND #PWR0302
+L power:GND #PWR0152
 U 1 1 5D194EBD
 P 10500 10500
-F 0 "#PWR0302" H 10500 10250 50  0001 C CNN
+F 0 "#PWR0152" H 10500 10250 50  0001 C CNN
 F 1 "GND" H 10505 10327 50  0000 C CNN
 F 2 "" H 10500 10500 50  0001 C CNN
@@
 	9650 1600 9650 2500
 $Comp
-L unlockoslo:GND_ETH #PWR0301
+L unlockoslo:GND_ETH #PWR0153
 U 1 1 5D7FEFF9
 P 3800 4200
-F 0 "#PWR0301" H 3800 3950 50  0001 C CNN
+F 0 "#PWR0153" H 3800 3950 50  0001 C CNN
 F 1 "GND_ETH" H 3805 4027 50  0000 C CNN
 F 2 "" H 3800 4200 50  0001 C CNN
@@
 Text HLabel 2000 3400 0    50   Input ~ 0
 Vin_B2
+$Comp
+L power:PWR_FLAG #FLG0104
+U 1 1 5D1A51B4
+P 5100 7750
+F 0 "#FLG0104" H 5100 7825 50  0001 C CNN
+F 1 "PWR_FLAG" H 5100 7923 50  0001 C CNN
+F 2 "" H 5100 7750 50  0001 C CNN
+F 3 "~" H 5100 7750 50  0001 C CNN
+	1    5100 7750
+	1    0    0    -1
+$EndComp
+Wire Wire Line
+	5100 7750 5100 7800
+Wire Wire Line
+	5100 7800 5000 7800
+Connection ~ 5000 7800
+$Comp
+L power:PWR_FLAG #FLG0105
+U 1 1 5D1BC100
+P 3900 3400
+F 0 "#FLG0105" H 3900 3475 50  0001 C CNN
+F 1 "PWR_FLAG" H 3900 3573 50  0001 C CNN
+F 2 "" H 3900 3400 50  0001 C CNN
+F 3 "~" H 3900 3400 50  0001 C CNN
+	1    3900 3400
+	1    0    0    -1
+$EndComp
+Wire Wire Line
+	3900 3400 3900 3500
+Connection ~ 3900 3500
+Wire Wire Line
+	3900 3500 4400 3500
 $EndSCHEMATC

Commit message: wip
Parts:
- D301, D302: footprint (none) -> Diodes_SMD:Diode_Bridge_TO-269AA
- Q301: footprint (none) -> Package_SO:SO-8_3.9x4.9mm_P1.27mm; symbol Device:Q_NMOS_DGS -> unlockoslo:Q_NMOS_SSSGDDDD
- Q302: footprint (none) -> Package_TO_SOT_SMD:SOT-23; symbol Device:Q_PMOS_DGS -> Device:Q_PMOS_GSD
- R311: value 0.12 -> 120m
Connections:
- net GND: now also Q302.2 (S); no longer Q302.3 (S)
- net at C315.2, TR301.2: now also Q301.5 (D), Q301.6 (D), Q301.7 (D), Q301.8 (D); no longer Q301.1 (D)
- net at Q302.1 (G): now also C312.1, D307.2 (A), R313.1; no longer C315.1
- net at Q301.2 (S): now also Q301.1 (S), Q301.3 (S), R307.2, R311.1; no longer R306.2
- new net: C315.1, Q302.3 (D)
- new net: Q301.4 (G), R306.2
Other:
- moved on the sheet: C317, C318, D308, R315, R316, R317, R318, U303
Changed lines of the file:
@@
 F 0 "D301" H 2600 1800 50  0000 L CNN
 F 1 "CDBHD1100L-G" H 2400 1900 50  0000 L CNN
-F 2 "" H 2700 1300 50  0001 C CNN
-F 3 "~" H 2700 1300 50  0001 C CNN
+F 2 "Diodes_SMD:Diode_Bridge_TO-269AA" H 2700 1300 50  0001 C CNN
+F 3 "http://www.comchiptech.com/admin/files/product/CDBHD140L-G%20Thru.%20CDBHD1100L-G%20RevC.PDF" H 2700 1300 50  0001 C CNN
 	1    2700 1300
 	1    0    0    -1
@@
 F 0 "D302" H 2600 3500 50  0000 L CNN
 F 1 "CDBHD1100L-G" H 2400 3600 50  0000 L CNN
-F 2 "" H 2700 3000 50  0001 C CNN
-F 3 "~" H 2700 3000 50  0001 C CNN
+F 2 "Diodes_SMD:Diode_Bridge_TO-269AA" H 2700 3000 50  0001 C CNN
+F 3 "http://www.comchiptech.com/admin/files/product/CDBHD140L-G%20Thru.%20CDBHD1100L-G%20RevC.PDF" H 2700 3000 50  0001 C CNN
 	1    2700 3000
 	1    0    0    -1
@@
 	5000 7700 5000 7300
 $Comp
-L Device:Q_PMOS_DGS Q302
+L Device:Q_PMOS_GSD Q302
 U 1 1 5CDBCD1F
 P 8400 6600
 F 0 "Q302" H 8606 6646 50  0000 L CNN
 F 1 "Si2325DS" H 8606 6555 50  0000 L CNN
-F 2 "" H 8600 6700 50  0001 C CNN
+F 2 "Package_TO_SOT_SMD:SOT-23" H 8600 6700 50  0001 C CNN
 F 3 "~" H 8400 6600 50  0001 C CNN
 	1    8400 6600
@@
 	8500 6300 8500 6400
 $Comp
-L Device:Q_NMOS_DGS Q301
+L unlockoslo:Q_NMOS_SSSGDDDD Q301
 U 1 1 5CE0FF51
 P 6700 5400
 F 0 "Q301" H 6906 5446 50  0000 L CNN
 F 1 "Si4848DY" H 6906 5355 50  0000 L CNN
-F 2 "" H 6900 5500 50  0001 C CNN
+F 2 "Package_SO:SO-8_3.9x4.9mm_P1.27mm" H 6900 5500 50  0001 C CNN
 F 3 "~" H 6700 5400 50  0001 C CNN
 	1    6700 5400
@@
 P 6800 5950
 F 0 "R311" H 6870 6041 50  0000 L CNN
-F 1 "0.12" H 6870 5950 50  0000 L CNN
+F 1 "120m" H 6870 5950 50  0000 L CNN
 F 2 "Resistor_SMD:R_0402_1005Metric" V 6730 5950 50  0001 C CNN
 F 3 "~" H 6800 5950 50  0001 C CNN
@@
 	5500 6600 6200 6600
 Wire Wire Line
-	6800 5200 6800 4800
+	6800 5200 6800 5100
 Text Label 6050 5400 2    50   ~ 0
 GATE
@@
 	7900 9000 7900 9700
 Wire Wire Line
-	8300 9300 8600 9300
-Wire Wire Line
-	10500 8800 10700 8800
-Connection ~ 10500 8800
-Wire Wire Line
-	10500 9300 10500 8800
-Wire Wire Line
-	9600 9700 9700 9700
-Wire Wire Line
-	9200 9300 9700 9300
-Wire Wire Line
-	9200 9700 9300 9700
-Connection ~ 9200 9700
-Wire Wire Line
-	9200 9300 9200 9700
-Wire Wire Line
-	10100 9700 10500 9700
-Connection ~ 10100 9700
-Wire Wire Line
-	10100 9300 10100 9700
-Wire Wire Line
-	10000 9300 10100 9300
+	8300 9300 8800 9300
+Wire Wire Line
+	10700 8800 10900 8800
+Connection ~ 10700 8800
+Wire Wire Line
+	10700 9300 10700 8800
+Wire Wire Line
+	9800 9700 9900 9700
+Wire Wire Line
+	9400 9300 9900 9300
+Wire Wire Line
+	9400 9700 9500 9700
+Connection ~ 9400 9700
+Wire Wire Line
+	9400 9300 9400 9700
+Wire Wire Line
+	10300 9700 10700 9700
+Connection ~ 10300 9700
+Wire Wire Line
+	10300 9300 10300 9700
+Wire Wire Line
+	10200 9300 10300 9300
 $Comp
 L Device:C C317
 U 1 1 5D28C6A9
-P 9850 9300
-F 0 "C317" V 9598 9300 50  0000 C CNN
-F 1 "10pF" V 9689 9300 50  0000 C CNN
-F 2 "Capacitor_SMD:C_0402_1005Metric" H 9888 9150 50  0001 C CNN
-F 3 "~" H 9850 9300 50  0001 C CNN
-	1    9850 9300
-	0    1    1    0
-$EndComp
-Wire Wire Line
-	10500 9700 10500 9900
-Connection ~ 10500 9700
-Wire Wire Line
-	10000 9700 10100 9700
-Wire Wire Line
-	8800 9700 9200 9700
+P 10050 9300
+F 0 "C317" V 9798 9300 50  0000 C CNN
+F 1 "10pF" V 9889 9300 50  0000 C CNN
+F 2 "Capacitor_SMD:C_0402_1005Metric" H 10088 9150 50  0001 C CNN
+F 3 "~" H 10050 9300 50  0001 C CNN
+	1    10050 9300
+	0    1    1    0
+$EndComp
+Wire Wire Line
+	10700 9700 10700 9900
+Connection ~ 10700 9700
+Wire Wire Line
+	10200 9700 10300 9700
+Wire Wire Line
+	9000 9700 9400 9700
 $Comp
 L Device:C C318
 U 1 1 5D24F557
-P 9850 9700
-F 0 "C318" V 9598 9700 50  0000 C CNN
-F 1 "15nF" V 9689 9700 50  0000 C CNN
-F 2 "Capacitor_SMD:C_0402_1005Metric" H 9888 9550 50  0001 C CNN
-F 3 "~" H 9850 9700 50  0001 C CNN
-	1    9850 9700
+P 10050 9700
+F 0 "C318" V 9798 9700 50  0000 C CNN
+F 1 "15nF" V 9889 9700 50  0000 C CNN
+F 2 "Capacitor_SMD:C_0402_1005Metric" H 10088 9550 50  0001 C CNN
+F 3 "~" H 10050 9700 50  0001 C CNN
+	1    10050 9700
 	0    1    1    0
 $EndComp
@@
 L Device:R R315
 U 1 1 5D24EE83
-P 9450 9700
-F 0 "R315" V 9657 9700 50  0000 C CNN
-F 1 "10k" V 9566 9700 50  0000 C CNN
-F 2 "Resistor_SMD:R_0402_1005Metric" V 9380 9700 50  0001 C CNN
-F 3 "~" H 9450 9700 50  0001 C CNN
-	1    9450 9700
+P 9650 9700
+F 0 "R315" V 9857 9700 50  0000 C CNN
+F 1 "10k" V 9766 9700 50  0000 C CNN
+F 2 "Resistor_SMD:R_0402_1005Metric" V 9580 9700 50  0001 C CNN
+F 3 "~" H 9650 9700 50  0001 C CNN
+	1    9650 9700
 	0    -1   -1   0
 $EndComp
 Wire Wire Line
-	8800 9700 8800 9600
-Connection ~ 8800 9700
-Wire Wire Line
-	7900 9700 8800 9700
-Connection ~ 10500 9900
-Wire Wire Line
-	10500 9600 10500 9700
+	9000 9700 9000 9600
+Connection ~ 9000 9700
+Wire Wire Line
+	7900 9700 9000 9700
+Connection ~ 10700 9900
+Wire Wire Line
+	10700 9600 10700 9700
 $Comp
 L Device:R R316
 U 1 1 5D1E0D58
-P 10500 9450
-F 0 "R316" H 10430 9404 50  0000 R CNN
-F 1 "41.2k" H 10430 9495 50  0000 R CNN
-F 2 "Resistor_SMD:R_0402_1005Metric" V 10430 9450 50  0001 C CNN
-F 3 "~" H 10500 9450 50  0001 C CNN
-	1    10500 9450
+P 10700 9450
+F 0 "R316" H 10630 9404 50  0000 R CNN
+F 1 "41.2k" H 10630 9495 50  0000 R CNN
+F 2 "Resistor_SMD:R_0402_1005Metric" V 10630 9450 50  0001 C CNN
+F 3 "~" H 10700 9450 50  0001 C CNN
+	1    10700 9450
 	-1   0    0    1
 $EndComp
 Wire Wire Line
-	8800 9800 8800 9700
-Wire Wire Line
-	10500 9900 10500 10000
-Wire Wire Line
-	8900 9900 10500 9900
-Connection ~ 8800 10400
-Wire Wire Line
-	8800 10400 8300 10400
-Wire Wire Line
-	10500 10400 10500 10300
-Connection ~ 10500 10400
-Wire Wire Line
-	8800 10400 8800 10000
-Wire Wire Line
-	10500 10400 8800 10400
-Wire Wire Line
-	10500 10500 10500 10400
+	9000 9800 9000 9700
+Wire Wire Line
+	10700 9900 10700 10000
+Wire Wire Line
+	9100 9900 10700 9900
+Connection ~ 9000 10400
+Wire Wire Line
+	9000 10400 8300 10400
+Wire Wire Line
+	10700 10400 10700 10300
+Connection ~ 10700 10400
+Wire Wire Line
+	9000 10400 9000 10000
+Wire Wire Line
+	10700 10400 9000 10400
+Wire Wire Line
+	10700 10500 10700 10400
 $Comp
 L Device:R R317
 U 1 1 5D197E47
-P 10500 10150
-F 0 "R317" H 10430 10104 50  0000 R CNN
-F 1 "11k" H 10430 10195 50  0000 R CNN
-F 2 "Resistor_SMD:R_0402_1005Metric" V 10430 10150 50  0001 C CNN
-F 3 "~" H 10500 10150 50  0001 C CNN
-	1    10500 10150
+P 10700 10150
+F 0 "R317" H 10630 10104 50  0000 R CNN
+F 1 "11k" H 10630 10195 50  0000 R CNN
+F 2 "Resistor_SMD:R_0402_1005Metric" V 10630 10150 50  0001 C CNN
+F 3 "~" H 10700 10150 50  0001 C CNN
+	1    10700 10150
 	-1   0    0    1
 $EndComp
@@
 L power:GND #PWR0152
 U 1 1 5D194EBD
-P 10500 10500
-F 0 "#PWR0152" H 10500 10250 50  0001 C CNN
-F 1 "GND" H 10505 10327 50  0000 C CNN
-F 2 "" H 10500 10500 50  0001 C CNN
-F 3 "" H 10500 10500 50  0001 C CNN
-	1    10500 10500
-	1    0    0    -1
-$EndComp
-Wire Wire Line
-	8800 8800 8800 9000
-Wire Wire Line
-	8300 8800 8800 8800
-Wire Wire Line
-	8800 8800 10500 8800
-Connection ~ 8800 8800
+P 10700 10500
+F 0 "#PWR0152" H 10700 10250 50  0001 C CNN
+F 1 "GND" H 10705 10327 50  0000 C CNN
+F 2 "" H 10700 10500 50  0001 C CNN
+F 3 "" H 10700 10500 50  0001 C CNN
+	1    10700 10500
+	1    0    0    -1
+$EndComp
+Wire Wire Line
+	9000 8800 9000 9000
+Wire Wire Line
+	8300 8800 9000 8800
+Wire Wire Line
+	9000 8800 10700 8800
+Connection ~ 9000 8800
 $Comp
 L Device:D_x2_Serial_ACK D308
 U 1 1 5D0EEC09
-P 8800 9300
-F 0 "D308" V 8846 9379 50  0000 L CNN
-F 1 "BAV99" V 8755 9379 50  0000 L CNN
-F 2 "Diode_SMD:D_SOT-23_ANK" H 8800 9300 50  0001 C CNN
-F 3 "~" H 8800 9300 50  0001 C CNN
-	1    8800 9300
+P 9000 9300
+F 0 "D308" V 9046 9379 50  0000 L CNN
+F 1 "BAV99" V 8955 9379 50  0000 L CNN
+F 2 "Diode_SMD:D_SOT-23_ANK" H 9000 9300 50  0001 C CNN
+F 3 "~" H 9000 9300 50  0001 C CNN
+	1    9000 9300
 	0    1    -1   0
 $EndComp
@@
 L Device:R R318
 U 1 1 5D0EBF76
-P 10850 8800
-F 0 "R318" V 10643 8800 50  0000 C CNN
-F 1 "49.9" V 10734 8800 50  0000 C CNN
-F 2 "Resistor_SMD:R_0402_1005Metric" V 10780 8800 50  0001 C CNN
-F 3 "~" H 10850 8800 50  0001 C CNN
-	1    10850 8800
+P 11050 8800
+F 0 "R318" V 10843 8800 50  0000 C CNN
+F 1 "49.9" V 10934 8800 50  0000 C CNN
+F 2 "Resistor_SMD:R_0402_1005Metric" V 10980 8800 50  0001 C CNN
+F 3 "~" H 11050 8800 50  0001 C CNN
+	1    11050 8800
 	0    1    1    0
 $EndComp
@@
 L Reference_Voltage:TL431D U303
 U 1 1 5D0E968E
-P 8800 9900
-F 0 "U303" V 8846 9831 50  0000 R CNN
-F 1 "TL431D" V 8755 9831 50  0000 R CNN
-F 2 "Package_SO:SOIC-8_3.9x4.9mm_P1.27mm" H 8800 9650 50  0001 C CIN
-F 3 "http://www.ti.com/lit/ds/symlink/tl431.pdf" H 8800 9900 50  0001 C CIN
-	1    8800 9900
+P 9000 9900
+F 0 "U303" V 9046 9831 50  0000 R CNN
+F 1 "TL431D" V 8955 9831 50  0000 R CNN
+F 2 "Package_SO:SOIC-8_3.9x4.9mm_P1.27mm" H 9000 9650 50  0001 C CIN
+F 3 "http://www.ti.com/lit/ds/symlink/tl431.pdf" H 9000 9900 50  0001 C CIN
+	1    9000 9900
 	0    1    -1   0
 $EndComp
@@
 	15650 1300 15650 8800
 Wire Wire Line
-	11000 8800 15650 8800
+	11200 8800 15650 8800
 Text HLabel 15750 1300 2    50   Output ~ 0
 Vout
@@
 Wire Wire Line
 	3900 3500 4400 3500
+Wire Wire Line
+	6800 5700 6900 5700
+Wire Wire Line
+	6900 5700 6900 5600
+Wire Wire Line
+	6900 5700 7000 5700
+Wire Wire Line
+	7000 5700 7000 5600
+Connection ~ 6900 5700
+Wire Wire Line
+	6900 5200 6900 5100
+Wire Wire Line
+	6900 5100 6800 5100
+Connection ~ 6800 5100
+Wire Wire Line
+	6800 5100 6800 4800
+Wire Wire Line
+	7000 5200 7000 5100
+Wire Wire Line
+	7000 5100 6900 5100
+Connection ~ 6900 5100
+Wire Wire Line
+	7100 5200 7100 5100
+Wire Wire Line
+	7100 5100 7000 5100
+Connection ~ 7000 5100
 $EndSCHEMATC

Commit message: wip
Parts:
- U301: footprint (none) -> Package_SO:HTSSOP-20-1EP_4.4x6.5mm_P0.65mm_EP3.4x6.5mm_Mask2.4x3.7mm
Changed lines of the file:
@@
 F 0 "U301" H 4750 6400 50  0000 L CNN
 F 1 "TPS23754" H 4600 6300 50  0000 L CNN
-F 2 "" H 4800 6400 50  0001 C CNN
+F 2 "Package_SO:HTSSOP-20-1EP_4.4x6.5mm_P0.65mm_EP3.4x6.5mm_Mask2.4x3.7mm" H 4800 6400 50  0001 C CNN
 F 3 "" H 4800 6400 50  0001 C CNN
 	1    4800 6400
