File: pcb/base-1.0/poe.sch (KiCad schematic (older format))
At the start: 69 parts, among them Q301 Si4848DY, Q302 Si2325DS, Q303 Si7852DP, Q304 MMBTA06, Q305 MMBTA06, Q306 Si4850EY, U301 TPS23754, U302 FOD817AS, U303 TL431D

Commit message: wip
Parts:
- D305, D306, D307, D309, D311: footprint Diode_SMD:D_SOT-23_ANK -> Diode_SMD:D_SOD-323; mpn (none) -> BAS16HT3G
- D308: footprint Diode_SMD:D_SOT-23_ANK -> Package_TO_SOT_SMD:SOT-23; symbol Device:D_x2_Serial_ACK -> Device:D_x2_Serial_AKC
- D310, D312: footprint (none) -> Diode_SMD:D_SOT-23_ANK; mpn (none) -> BZX84C12LT1G
- TR301: value TRANSF6 -> PA2649NL; footprint (none) -> PAxxxxNL:PAxxxxNL
- U302: footprint Package_DIP:DIP-4_W7.62mm -> Package_DIP:SMDIP-4_W9.53mm; mpn (none) -> FOD817ASD
Connections:
- net at R312.1, R314.2, R316.2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: now also D308.2 (K); no longer D308.3 (K)
- net at C314.1, R314.1: now also D308.3 (common); no longer D308.2 (common)
Changed lines of the file:
@@
 P 9800 1600
 F 0 "TR301" H 9800 2082 50  0000 C CNN
-F 1 "TRANSF6" H 9800 1991 50  0000 C CNN
-F 2 "" H 9800 1600 50  0001 C CNN
-F 3 "" H 9800 1600 50  0001 C CNN
+F 1 "PA2649NL" H 9800 1991 50  0000 C CNN
+F 2 "PAxxxxNL:PAxxxxNL" H 9800 1600 50  0001 C CNN
+F 3 "http://productfinder.pulseeng.com/products/datasheets/P675.pdf" H 9800 1600 50  0001 C CNN
 	1    9800 1600
 	1    0    0    -1
@@
 F 0 "D312" V 13254 2629 50  0000 L CNN
 F 1 "12V" V 13345 2629 50  0000 L CNN
-F 2 "" H 13300 2550 50  0001 C CNN
-F 3 "~" H 13300 2550 50  0001 C CNN
+F 2 "Diode_SMD:D_SOT-23_ANK" H 13300 2550 50  0001 C CNN
+F 3 "https://www.onsemi.com/pub/Collateral/BZX84C2V4LT1-D.PDF" H 13300 2550 50  0001 C CNN
+F 4 "BZX84C12LT1G" H 13300 2550 50  0001 C CNN "mpn"
 	1    13300 2550
 	0    1    1    0
@@
 F 0 "D311" H 13250 1716 50  0000 C CNN
 F 1 "BAS16" H 13250 1625 50  0000 C CNN
-F 2 "Diode_SMD:D_SOT-23_ANK" H 13250 1500 50  0001 C CNN
-F 3 "~" H 13250 1500 50  0001 C CNN
+F 2 "Diode_SMD:D_SOD-323" H 13250 1500 50  0001 C CNN
+F 3 "http://www.onsemi.com/pub/Collateral/BAS16HT1-D.PDF" H 13250 1500 50  0001 C CNN
+F 4 "BAS16HT3G" H 13250 1500 50  0001 C CNN "mpn"
 	1    13250 1500
 	1    0    0    -1
@@
 F 0 "D309" V 10654 1629 50  0000 L CNN
 F 1 "BAS16" V 10745 1629 50  0000 L CNN
-F 2 "Diode_SMD:D_SOT-23_ANK" H 10700 1550 50  0001 C CNN
-F 3 "~" H 10700 1550 50  0001 C CNN
+F 2 "Diode_SMD:D_SOD-323" H 10700 1550 50  0001 C CNN
+F 3 "http://www.onsemi.com/pub/Collateral/BAS16HT1-D.PDF" H 10700 1550 50  0001 C CNN
+F 4 "BAS16HT3G" H 10700 1550 50  0001 C CNN "mpn"
 	1    10700 1550
 	0    1    1    0
@@
 F 0 "D310" V 11554 2629 50  0000 L CNN
 F 1 "12V" V 11645 2629 50  0000 L CNN
-F 2 "" H 11600 2550 50  0001 C CNN
-F 3 "~" H 11600 2550 50  0001 C CNN
+F 2 "Diode_SMD:D_SOT-23_ANK" H 11600 2550 50  0001 C CNN
+F 3 "https://www.onsemi.com/pub/Collateral/BZX84C2V4LT1-D.PDF" H 11600 2550 50  0001 C CNN
+F 4 "BZX84C12LT1G" H 11600 2550 50  0001 C CNN "mpn"
 	1    11600 2550
 	0    1    1    0
@@
 F 0 "D307" V 7746 6771 50  0000 R CNN
 F 1 "BAS16" V 7655 6771 50  0000 R CNN
-F 2 "Diode_SMD:D_SOT-23_ANK" H 7700 6850 50  0001 C CNN
-F 3 "~" H 7700 6850 50  0001 C CNN
+F 2 "Diode_SMD:D_SOD-323" H 7700 6850 50  0001 C CNN
+F 3 "http://www.onsemi.com/pub/Collateral/BAS16HT1-D.PDF" H 7700 6850 50  0001 C CNN
+F 4 "BAS16HT3G" H 7700 6850 50  0001 C CNN "mpn"
 	1    7700 6850
 	0    -1   -1   0
@@
 F 0 "D305" V 7054 7829 50  0000 L CNN
 F 1 "BAS16" V 7145 7829 50  0000 L CNN
-F 2 "Diode_SMD:D_SOT-23_ANK" H 7100 7750 50  0001 C CNN
-F 3 "~" H 7100 7750 50  0001 C CNN
+F 2 "Diode_SMD:D_SOD-323" H 7100 7750 50  0001 C CNN
+F 3 "http://www.onsemi.com/pub/Collateral/BAS16HT1-D.PDF" H 7100 7750 50  0001 C CNN
+F 4 "BAS16HT3G" H 7100 7750 50  0001 C CNN "mpn"
 	1    7100 7750
 	0    1    1    0
@@
 F 0 "D306" H 7350 7716 50  0000 C CNN
 F 1 "BAS16" H 7350 7625 50  0000 C CNN
-F 2 "Diode_SMD:D_SOT-23_ANK" H 7350 7500 50  0001 C CNN
-F 3 "~" H 7350 7500 50  0001 C CNN
+F 2 "Diode_SMD:D_SOD-323" H 7350 7500 50  0001 C CNN
+F 3 "http://www.onsemi.com/pub/Collateral/BAS16HT1-D.PDF" H 7350 7500 50  0001 C CNN
+F 4 "BAS16HT3G" H 7350 7500 50  0001 C CNN "mpn"
 	1    7350 7500
 	1    0    0    -1
@@
 F 0 "U302" H 7500 9225 50  0000 C CNN
 F 1 "FOD817AS" H 7500 9134 50  0000 C CNN
-F 2 "Package_DIP:DIP-4_W7.62mm" H 7300 8700 50  0001 L CIN
-F 3 "http://www.soselectronic.cz/a_info/resource/d/pc817.pdf" H 7500 8900 50  0001 L CNN
+F 2 "Package_DIP:SMDIP-4_W9.53mm" H 7300 8700 50  0001 L CIN
+F 3 "https://www.onsemi.com/pub/Collateral/FOD814-D.PDF" H 7500 8900 50  0001 L CNN
+F 4 "FOD817ASD	" H 7500 8900 50  0001 C CNN "mpn"
 	1    7500 8900
 	-1   0    0    -1
@@
 Connection ~ 9000 8800
 $Comp
-L Device:D_x2_Serial_ACK D308
+L Device:D_x2_Serial_AKC D308
 U 1 1 5D0EEC09
 P 9000 9300
 F 0 "D308" V 9046 9379 50  0000 L CNN
 F 1 "BAV99" V 8955 9379 50  0000 L CNN
-F 2 "Diode_SMD:D_SOT-23_ANK" H 9000 9300 50  0001 C CNN
+F 2 "Package_TO_SOT_SMD:SOT-23" H 9000 9300 50  0001 C CNN
 F 3 "~" H 9000 9300 50  0001 C CNN
 	1    9000 9300
@@
 Wire Wire Line
 	9250 1600 9600 1600
-Wire Wire Line
-	9650 1600 9650 2500
 $Comp
 L unlockoslo:GND_ETH #PWR0153
@@
 Wire Wire Line
 	3800 3700 3800 3500
-Connection ~ 9650 2500
 Wire Wire Line
 	8500 4800 8500 1500
