File: pcb/base-1.0/poe.sch (KiCad schematic (older format))
At the start: 69 parts, among them Q301 Si4848DY, Q302 Si2325DS, Q303 Si7852DP, Q304 MMBTA06, Q305 MMBTA06, Q306 Si4850EY, U301 TPS23754, U302 FOD817AS, U303 TL431D

Commit message: wip
Parts:
- D301, D302: footprint Diodes_SMD:Diode_Bridge_TO-269AA -> Package_TO_SOT_SMD:TO-269AA
- FB301, FB302: footprint Inductor_SMD:L_0603_1608Metric -> Inductor_SMD:L_1206_3216Metric
- L301: footprint (none) -> 74404043102A:74404043102A
- L302: footprint (none) -> 744043003:744043003; mpn (none) -> 744043003
- L303: mpn (none) -> 744770122
Other:
- moved on the sheet: C316, C319, C320, C321, D309, D310, D311, D312, Q303, Q304, Q305, Q306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

Commit message: wip
Parts:
- L303: footprint (none) -> 744770122:744770122
- Q303: footprint (none) -> Package_SO:PowerPAK_SO-8_Single
- Q304, Q305: footprint (none) -> Package_TO_SOT_SMD:SOT-23
- Q306: footprint (none) -> Package_SO:PowerIntegrations_SO-8
Changed lines of the file:
@@
 F 0 "Q306" H 14106 2046 50  0000 L CNN
 F 1 "Si4850EY" H 14106 1955 50  0000 L CNN
-F 2 "" H 14100 2100 50  0001 C CNN
-F 3 "~" H 13900 2000 50  0001 C CNN
+F 2 "Package_SO:PowerIntegrations_SO-8" H 14100 2100 50  0001 C CNN
+F 3 "http://www.vishay.com/docs/71146/71146.pdf" H 13900 2000 50  0001 C CNN
 	1    13900 2000
 	1    0    0    -1
@@
 F 0 "L303" V 14575 1300 50  0000 C CNN
 F 1 "22uH" V 14484 1300 50  0000 C CNN
-F 2 "" H 14350 1300 50  0001 C CNN
+F 2 "744770122:744770122" H 14350 1300 50  0001 C CNN
 F 3 "https://katalog.we-online.de/pbs/datasheet/744770122.pdf" H 14350 1300 50  0001 C CNN
 F 4 "744770122" V 14350 1300 50  0001 C CNN "mpn"
@@
 F 0 "Q305" V 13628 2100 50  0000 C CNN
 F 1 "MMBTA06" V 13537 2100 50  0000 C CNN
-F 2 "" H 13500 2200 50  0001 C CNN
-F 3 "~" H 13300 2100 50  0001 C CNN
+F 2 "Package_TO_SOT_SMD:SOT-23" H 13500 2200 50  0001 C CNN
+F 3 "https://www.mccsemi.com/pdf/Products/MMBTA05-MMBTA06(SOT-23).PDF" H 13300 2100 50  0001 C CNN
 	1    13300 2100
 	0    -1   -1   0
@@
 F 0 "Q303" V 11451 2800 50  0000 C CNN
 F 1 "Si7852DP" V 11542 2800 50  0000 C CNN
-F 2 "" H 11400 2900 50  0001 C CNN
-F 3 "~" H 11200 2800 50  0001 C CNN
+F 2 "Package_SO:PowerPAK_SO-8_Single" H 11400 2900 50  0001 C CNN
+F 3 "http://www.vishay.com/docs/71627/si7852dp.pdf" H 11200 2800 50  0001 C CNN
 	1    11200 2800
 	0    1    1    0
@@
 F 0 "Q304" H 11491 1946 50  0000 L CNN
 F 1 "MMBTA06" H 11491 1855 50  0000 L CNN
-F 2 "" H 11500 2000 50  0001 C CNN
-F 3 "~" H 11300 1900 50  0001 C CNN
+F 2 "Package_TO_SOT_SMD:SOT-23" H 11500 2000 50  0001 C CNN
+F 3 "https://www.mccsemi.com/pdf/Products/MMBTA05-MMBTA06(SOT-23).PDF" H 11300 1900 50  0001 C CNN
 	1    11300 1900
 	-1   0    0    -1

Commit message: wip
Changed lines of the file:
@@
 	3300 5100 4600 5100
 Wire Wire Line
-	15650 1300 15650 8900
+	15650 1300 15650 8800
 Wire Wire Line
-	11200 8800 15650 8900
+	11200 8800 15650 8800
 Text HLabel 15750 1300 2    50   Output ~ 0
 Vout

Commit message: o Replacing footprints with IPC footprints.
Parts:
- C301, C302, C303, C304, C305, C306, C307, C308, C309, C310, C311, C312, C313, C314, C315, C316, C317, C318, C319, C320, C321: footprint Capacitor_SMD:C_0402_1005Metric -> IPC-7351-CAPC:CAPC_1005x015
- R301, R302, R303, R304, R305, R306, R307, R308, R309, R310, R311, R312, R313, R314, R315, R316, R317, R318, R319, R320: footprint Resistor_SMD:R_0402_1005Metric -> IPC-7351-RESC:RESC_1005x015

Commit message: o More values.
Parts:
- C314: value C -> 1uF
Changed lines of the file:
@@
 F 1 "TPS23754" H 4600 6300 50  0000 L CNN
 F 2 "Package_SO:HTSSOP-20-1EP_4.4x6.5mm_P0.65mm_EP3.4x6.5mm_Mask2.4x3.7mm" H 4800 6400 50  0001 C CNN
-F 3 "" H 4800 6400 50  0001 C CNN
+F 3 "http://www.ti.com/lit/ds/symlink/tps23754.pdf" H 4800 6400 50  0001 C CNN
 	1    4800 6400
 	1    0    0    -1
@@
 P 8300 9950
 F 0 "C314" H 8415 9996 50  0000 L CNN
-F 1 "C" H 8415 9905 50  0000 L CNN
+F 1 "1uF" H 8415 9905 50  0000 L CNN
 F 2 "IPC-7351-CAPC:CAPC_1005x015" H 8338 9800 50  0001 C CNN
 F 3 "~" H 8300 9950 50  0001 C CNN

Commit message: o More values.
Parts:
- R313: value R -> 10k
Changed lines of the file:
@@
 P 8100 6850
 F 0 "R313" H 8170 6896 50  0000 L CNN
-F 1 "R" H 8170 6805 50  0000 L CNN
+F 1 "10k" H 8170 6805 50  0000 L CNN
 F 2 "IPC-7351-RESC:RESC_1005x015" V 8030 6850 50  0001 C CNN
 F 3 "~" H 8100 6850 50  0001 C CNN

Commit message: o Selecting parts.
Parts:
- C301: mpn (none) -> C1812C102KGRACAUTO
- C302, C303: mpn (none) -> CL21B104KCFNNNE
- C304, C305, C307, C312, C314: mpn (none) -> CL05A105MQ5NNNC
- C306, C313: footprint IPC-7351-CAPC:CAPC_1005x015 -> IPC-7351-CAPC:CAPC_3216x040; mpn (none) -> CL31B105KCHNFNE
- C310: mpn (none) -> CL05B223KP5NNNC
- C315: mpn (none) -> CL31B473KEHNNNE
- C316: mpn (none) -> CL05B222KB5NNNC
- C317: mpn (none) -> CL05C100JB5NNNC
- C318: mpn (none) -> CL05B153KO5NNNC
- C319: mpn (none) -> CL05C101JB5NNNC
- R304: Tolerance (none) -> 1%; Tollerance 1% -> (none)

Commit message: o Selecting parts.
Parts:
- C308: footprint IPC-7351-CAPC:CAPC_1005x015 -> IPC-7351-CAPC:CAPC_3216x040; mpn (none) -> CL31A226KAHNNNE
- C309, C311: footprint IPC-7351-CAPC:CAPC_1005x015 -> Capacitor_SMD:C_Elec_8x10.2; mpn (none) -> UUX2A220MNL6GS
- C320: footprint IPC-7351-CAPC:CAPC_1005x015 -> Capacitor_SMD:CP_Elec_8x10; mpn (none) -> EEE-1EA101AP
- C321: footprint IPC-7351-CAPC:CAPC_1005x015 -> Capacitor_SMD:CP_Elec_5x5.4; mpn (none) -> 865080442004
- Q301: mpn (none) -> SI4848DY-T1-E3
- Q302: mpn (none) -> SI2325DS-T1-E3
- Q303: mpn (none) -> SI7852DP-T1-E3
- Q304, Q305: mpn (none) -> MMBTA06-TP
- Q306: mpn (none) -> SI4850EY-T1-E3
Changed lines of the file:
@@
 F 2 "Package_SO:PowerIntegrations_SO-8" H 14100 2100 50  0001 C CNN
 F 3 "http://www.vishay.com/docs/71146/71146.pdf" H 13900 2000 50  0001 C CNN
+F 4 "SI4850EY-T1-E3" H 13900 2000 50  0001 C CNN "mpn"
 	1    13900 2000
 	1    0    0    -1
@@
 F 2 "Package_TO_SOT_SMD:SOT-23" H 13500 2200 50  0001 C CNN
 F 3 "https://www.mccsemi.com/pdf/Products/MMBTA05-MMBTA06(SOT-23).PDF" H 13300 2100 50  0001 C CNN
+F 4 "MMBTA06-TP" H 13300 2100 50  0001 C CNN "mpn"
 	1    13300 2100
 	0    -1   -1   0
@@
 F 0 "C320" H 14815 2141 50  0000 L CNN
 F 1 "100uF" H 14815 2050 50  0000 L CNN
-F 2 "IPC-7351-CAPC:CAPC_1005x015" H 14738 1900 50  0001 C CNN
-F 3 "~" H 14700 2050 50  0001 C CNN
+F 2 "Capacitor_SMD:CP_Elec_8x10" H 14738 1900 50  0001 C CNN
+F 3 "https://industrial.panasonic.com/cdbs/www-data/pdf/RDE0000/ABA0000C1142.pdf" H 14700 2050 50  0001 C CNN
 F 4 "16V" H 14815 1959 50  0000 L CNN "Voltage"
+F 5 "EEE-1EA101AP" H 14700 2050 50  0001 C CNN "mpn"
 	1    14700 2050
 	1    0    0    -1
@@
 F 0 "C321" H 15365 2141 50  0000 L CNN
 F 1 "22uF" H 15365 2050 50  0000 L CNN
-F 2 "IPC-7351-CAPC:CAPC_1005x015" H 15288 1900 50  0001 C CNN
-F 3 "~" H 15250 2050 50  0001 C CNN
+F 2 "Capacitor_SMD:CP_Elec_5x5.4" H 15288 1900 50  0001 C CNN
+F 3 "https://katalog.we-online.de/pbs/datasheet/865080442004.pdf" H 15250 2050 50  0001 C CNN
 F 4 "16V" H 15365 1959 50  0000 L CNN "Voltage"
+F 5 "865080442004" H 15250 2050 50  0001 C CNN "mpn"
 	1    15250 2050
 	1    0    0    -1
@@
 F 2 "Package_SO:PowerPAK_SO-8_Single" H 11400 2900 50  0001 C CNN
 F 3 "http://www.vishay.com/docs/71627/si7852dp.pdf" H 11200 2800 50  0001 C CNN
+F 4 "SI7852DP-T1-E3" H 11200 2800 50  0001 C CNN "mpn"
 	1    11200 2800
 	0    1    1    0
@@
 F 2 "Package_TO_SOT_SMD:SOT-23" H 11500 2000 50  0001 C CNN
 F 3 "https://www.mccsemi.com/pdf/Products/MMBTA05-MMBTA06(SOT-23).PDF" H 11300 1900 50  0001 C CNN
+F 4 "MMBTA06-TP" H 11300 1900 50  0001 C CNN "mpn"
 	1    11300 1900
 	-1   0    0    -1
@@
 F 0 "C309" H 6815 1641 50  0000 L CNN
 F 1 "22uF" H 6815 1550 50  0000 L CNN
-F 2 "IPC-7351-CAPC:CAPC_1005x015" H 6738 1400 50  0001 C CNN
+F 2 "Capacitor_SMD:C_Elec_8x10.2" H 6738 1400 50  0001 C CNN
 F 3 "~" H 6700 1550 50  0001 C CNN
 F 4 "100V" H 6815 1459 50  0000 L CNN "Voltage"
+F 5 "UUX2A220MNL6GS" H 6700 1550 50  0001 C CNN "mpn"
 	1    6700 1550
 	1    0    0    -1
@@
 F 0 "C311" H 7315 1641 50  0000 L CNN
 F 1 "22uF" H 7315 1550 50  0000 L CNN
-F 2 "IPC-7351-CAPC:CAPC_1005x015" H 7238 1400 50  0001 C CNN
+F 2 "Capacitor_SMD:C_Elec_8x10.2" H 7238 1400 50  0001 C CNN
 F 3 "~" H 7200 1550 50  0001 C CNN
 F 4 "100V" H 7315 1459 50  0000 L CNN "Voltage"
+F 5 "UUX2A220MNL6GS" H 7200 1550 50  0001 C CNN "mpn"
 	1    7200 1550
 	1    0    0    -1
@@
 F 1 "Si2325DS" H 8606 6555 50  0000 L CNN
 F 2 "Package_TO_SOT_SMD:SOT-23" H 8600 6700 50  0001 C CNN
-F 3 "~" H 8400 6600 50  0001 C CNN
+F 3 "http://www.vishay.com/docs/73238/73238.pdf" H 8400 6600 50  0001 C CNN
+F 4 "SI2325DS-T1-E3" H 8400 6600 50  0001 C CNN "mpn"
 	1    8400 6600
 	1    0    0    -1
@@
 F 1 "Si4848DY" H 6906 5355 50  0000 L CNN
 F 2 "Package_SO:SO-8_3.9x4.9mm_P1.27mm" H 6900 5500 50  0001 C CNN
-F 3 "~" H 6700 5400 50  0001 C CNN
+F 3 "http://www.vishay.com/docs/71356/71356.pdf" H 6700 5400 50  0001 C CNN
+F 4 "SI4848DY-T1-E3" H 6700 5400 50  0001 C CNN "mpn"
 	1    6700 5400
 	1    0    0    -1
@@
 F 0 "C308" H 6715 7841 50  0000 L CNN
 F 1 "22uF" H 6715 7750 50  0000 L CNN
-F 2 "IPC-7351-CAPC:CAPC_1005x015" H 6638 7600 50  0001 C CNN
+F 2 "IPC-7351-CAPC:CAPC_3216x040" H 6638 7600 50  0001 C CNN
 F 3 "~" H 6600 7750 50  0001 C CNN
 F 4 "25V" H 6715 7659 50  0000 L CNN "Voltage"
+F 5 "CL31A226KAHNNNE" H 6600 7750 50  0001 C CNN "mpn"
 	1    6600 7750
 	1    0    0    -1
