File: pcb/base-1.0/poe.sch (KiCad schematic (older format))
At the start: 69 parts, among them Q301 Si4848DY, Q302 Si2325DS, Q303 Si7852DP, Q304 MMBTA06, Q305 MMBTA06, Q306 Si4850EY, U301 TPS23754, U302 FOD817AS, U303 TL431D

Commit message: o More part numbers.
Parts:
- D301, D302: mpn (none) -> CDBHD1100L-G
- D303, D304: mpn (none) -> SMAJ58A
Changed lines of the file:
@@
 F 2 "Package_TO_SOT_SMD:TO-269AA" H 2700 1300 50  0001 C CNN
 F 3 "http://www.comchiptech.com/admin/files/product/CDBHD140L-G%20Thru.%20CDBHD1100L-G%20RevC.PDF" H 2700 1300 50  0001 C CNN
+F 4 "CDBHD1100L-G" H 2700 1300 50  0001 C CNN "mpn"
 	1    2700 1300
 	1    0    0    -1
@@
 F 2 "Package_TO_SOT_SMD:TO-269AA" H 2700 3000 50  0001 C CNN
 F 3 "http://www.comchiptech.com/admin/files/product/CDBHD140L-G%20Thru.%20CDBHD1100L-G%20RevC.PDF" H 2700 3000 50  0001 C CNN
+F 4 "CDBHD1100L-G" H 2700 3000 50  0001 C CNN "mpn"
 	1    2700 3000
 	1    0    0    -1
@@
 F 3 "~" H 3800 2250 50  0001 C CNN
 F 4 "58V" V 3891 2329 50  0000 L CNN "Voltage"
+F 5 "SMAJ58A" V 3800 2250 50  0001 C CNN "mpn"
 	1    3800 2250
 	0    1    1    0
@@
 F 2 "Diode_SMD:D_SMA" H 3800 3850 50  0001 C CNN
 F 3 "~" H 3800 3850 50  0001 C CNN
+F 4 "SMAJ58A" V 3800 3850 50  0001 C CNN "mpn"
 	1    3800 3850
 	0    -1   -1   0

Commit message: o Finding more components. o Refreshing generated files.
Parts:
- D308: mpn (none) -> BAV99,235
Changed lines of the file:
@@
 F 2 "Package_TO_SOT_SMD:SOT-23" H 9000 9300 50  0001 C CNN
 F 3 "~" H 9000 9300 50  0001 C CNN
+F 4 "BAV99,235" V 9000 9300 50  0001 C CNN "mpn"
 	1    9000 9300
 	0    1    -1   0

Commit message: o Selecting more parts, fixing footprints.
Parts:
- C301: footprint IPC-7351-CAPC:CAPC_1005x015 -> IPC-7351-CAPC:CAPC_4532x040
- C302, C303: footprint IPC-7351-CAPC:CAPC_1005x015 -> IPC-7351-CAPC:CAPC_2012x040
- C315: footprint IPC-7351-CAPC:CAPC_1005x015 -> IPC-7351-CAPC:CAPC_3216x040
- C320: footprint Capacitor_SMD:CP_Elec_8x10 -> Capacitor_SMD:CP_Elec_8x10.2
- FB301, FB302: value Ferrite_Bead -> 500; mpn (none) -> MI1206L501R-10
Changed lines of the file:
@@
 F 0 "C320" H 14815 2141 50  0000 L CNN
 F 1 "100uF" H 14815 2050 50  0000 L CNN
-F 2 "Capacitor_SMD:CP_Elec_8x10" H 14738 1900 50  0001 C CNN
+F 2 "Capacitor_SMD:CP_Elec_8x10.2" H 14738 1900 50  0001 C CNN
 F 3 "https://industrial.panasonic.com/cdbs/www-data/pdf/RDE0000/ABA0000C1142.pdf" H 14700 2050 50  0001 C CNN
 F 4 "16V" H 14815 1959 50  0000 L CNN "Voltage"
@@
 F 0 "C301" H 3415 2341 50  0000 L CNN
 F 1 "1nF" H 3415 2250 50  0000 L CNN
-F 2 "IPC-7351-CAPC:CAPC_1005x015" H 3338 2100 50  0001 C CNN
+F 2 "IPC-7351-CAPC:CAPC_4532x040" H 3338 2100 50  0001 C CNN
 F 3 "~" H 3300 2250 50  0001 C CNN
 F 4 "100V" H 3415 2159 50  0000 L CNN "Voltage"
@@
 P 3550 1300
 F 0 "FB301" V 3276 1300 50  0000 C CNN
-F 1 "Ferrite_Bead" V 3367 1300 50  0000 C CNN
+F 1 "500" V 3367 1300 50  0000 C CNN
 F 2 "Inductor_SMD:L_1206_3216Metric" V 3480 1300 50  0001 C CNN
 F 3 "~" H 3550 1300 50  0001 C CNN
+F 4 "MI1206L501R-10" V 3550 1300 50  0001 C CNN "mpn"
 	1    3550 1300
 	0    1    1    0
@@
 F 0 "C303" H 5815 1641 50  0000 L CNN
 F 1 "100nF" H 5815 1550 50  0000 L CNN
-F 2 "IPC-7351-CAPC:CAPC_1005x015" H 5738 1400 50  0001 C CNN
+F 2 "IPC-7351-CAPC:CAPC_2012x040" H 5738 1400 50  0001 C CNN
 F 3 "~" H 5700 1550 50  0001 C CNN
 F 4 "100V" H 5815 1459 50  0000 L CNN "Voltage"
@@
 F 0 "C302" H 4515 2341 50  0000 L CNN
 F 1 "100nF" H 4515 2250 50  0000 L CNN
-F 2 "IPC-7351-CAPC:CAPC_1005x015" H 4438 2100 50  0001 C CNN
+F 2 "IPC-7351-CAPC:CAPC_2012x040" H 4438 2100 50  0001 C CNN
 F 3 "~" H 4400 2250 50  0001 C CNN
 F 4 "100V" H 4515 2159 50  0000 L CNN "Voltage"
@@
 F 0 "C315" H 8385 6059 50  0000 R CNN
 F 1 "47nF" H 8385 6150 50  0000 R CNN
-F 2 "IPC-7351-CAPC:CAPC_1005x015" H 8538 6000 50  0001 C CNN
+F 2 "IPC-7351-CAPC:CAPC_3216x040" H 8538 6000 50  0001 C CNN
 F 3 "~" H 8500 6150 50  0001 C CNN
 F 4 "250V" H 8385 6241 50  0000 R CNN "Voltage"
@@
 P 3550 3500
 F 0 "FB302" V 3276 3500 50  0000 C CNN
-F 1 "Ferrite_Bead" V 3367 3500 50  0000 C CNN
+F 1 "500" V 3367 3500 50  0000 C CNN
 F 2 "Inductor_SMD:L_1206_3216Metric" V 3480 3500 50  0001 C CNN
 F 3 "~" H 3550 3500 50  0001 C CNN
+F 4 "MI1206L501R-10" V 3550 3500 50  0001 C CNN "mpn"
 	1    3550 3500
 	0    1    1    0

Commit message: o Improving footprints.
Parts:
- C309, C311: footprint Capacitor_SMD:C_Elec_8x10.2 -> Capacitor_SMD:CP_Elec_8x10.2
Changed lines of the file:
@@
 F 0 "C309" H 6815 1641 50  0000 L CNN
 F 1 "22uF" H 6815 1550 50  0000 L CNN
-F 2 "Capacitor_SMD:C_Elec_8x10.2" H 6738 1400 50  0001 C CNN
+F 2 "Capacitor_SMD:CP_Elec_8x10.2" H 6738 1400 50  0001 C CNN
 F 3 "~" H 6700 1550 50  0001 C CNN
 F 4 "100V" H 6815 1459 50  0000 L CNN "Voltage"
@@
 F 0 "C311" H 7315 1641 50  0000 L CNN
 F 1 "22uF" H 7315 1550 50  0000 L CNN
-F 2 "Capacitor_SMD:C_Elec_8x10.2" H 7238 1400 50  0001 C CNN
+F 2 "Capacitor_SMD:CP_Elec_8x10.2" H 7238 1400 50  0001 C CNN
 F 3 "~" H 7200 1550 50  0001 C CNN
 F 4 "100V" H 7315 1459 50  0000 L CNN "Voltage"

Commit message: o More footprints and mpns.
Parts:
- TR301: mpn (none) -> PA2649NL
Changed lines of the file:
@@
 F 2 "PAxxxxNL:PAxxxxNL" H 9800 1600 50  0001 C CNN
 F 3 "http://productfinder.pulseeng.com/products/datasheets/P675.pdf" H 9800 1600 50  0001 C CNN
+F 4 "PA2649NL" H 9800 1600 50  0001 C CNN "mpn"
 	1    9800 1600
 	1    0    0    -1

Commit message: o Adding IO extender for RPI header. o Adding mounting holes in schematic and PCB. o Fixing bad footprint: Capacitor_SMD:CP_Elec_8x10.2 => Capacitor_SMD:CP_Elec_8x10.
Parts:
- C309, C311, C320: footprint Capacitor_SMD:CP_Elec_8x10.2 -> Capacitor_SMD:CP_Elec_8x10
Connections:
- no-connect marks 0 -> 1
Changed lines of the file:
@@
 F 0 "C320" H 14815 2141 50  0000 L CNN
 F 1 "100uF" H 14815 2050 50  0000 L CNN
-F 2 "Capacitor_SMD:CP_Elec_8x10.2" H 14738 1900 50  0001 C CNN
+F 2 "Capacitor_SMD:CP_Elec_8x10" H 14738 1900 50  0001 C CNN
 F 3 "https://industrial.panasonic.com/cdbs/www-data/pdf/RDE0000/ABA0000C1142.pdf" H 14700 2050 50  0001 C CNN
 F 4 "16V" H 14815 1959 50  0000 L CNN "Voltage"
@@
 F 0 "C309" H 6815 1641 50  0000 L CNN
 F 1 "22uF" H 6815 1550 50  0000 L CNN
-F 2 "Capacitor_SMD:CP_Elec_8x10.2" H 6738 1400 50  0001 C CNN
+F 2 "Capacitor_SMD:CP_Elec_8x10" H 6738 1400 50  0001 C CNN
 F 3 "~" H 6700 1550 50  0001 C CNN
 F 4 "100V" H 6815 1459 50  0000 L CNN "Voltage"
@@
 F 0 "C311" H 7315 1641 50  0000 L CNN
 F 1 "22uF" H 7315 1550 50  0000 L CNN
-F 2 "Capacitor_SMD:CP_Elec_8x10.2" H 7238 1400 50  0001 C CNN
+F 2 "Capacitor_SMD:CP_Elec_8x10" H 7238 1400 50  0001 C CNN
 F 3 "~" H 7200 1550 50  0001 C CNN
 F 4 "100V" H 7315 1459 50  0000 L CNN "Voltage"
@@
 	0    1    1    0
 $EndComp
+NoConn ~ 5500 5900
 $EndSCHEMATC

Commit message: o Starting on PCB. o Fixing minor issues in the schmatic while doing layout.
Parts:
- NT301: footprint NetTie:NetTie-4_SMD_Pad0.5mm -> NetTie:NetTie-3_SMD_Pad0.5mm
- R311: footprint IPC-7351-RESC:RESC_1005x015 -> IPC-7351-RESC:RESC_3216x040; mpn (none) -> RL1206FR-070R12L; power 12W -> 0.25W
- R319: footprint IPC-7351-RESC:RESC_1005x015 -> IPC-7351-RESC:RESC_3216x040
- TR301: symbol Transformer:TRANSF6 -> unlockoslo:PA2649NL
Connections:
- net GND_ETH: now also C303.2, C306.2, C309.2, C311.2, C313.2, NT301.1; no longer NT301.2
- net CTL: now reaches C310.1, R310.1, U301.1 (CTL), U302.4
- net ARTN: now reaches NT301.3, R301.2, R302.2, R305.2, U301.17 (APD), U301.8 (ARTN)
- net ARTN: no longer NT301.1, U301.9 (RTN)
- net VB: now reaches C304.1, R309.2, R310.2, U301.2 (Vb)
- net GAT2: now reaches R308.2, U301.7 (GAT2)
- net T_POS: now reaches C319.1, D309.1 (K), L303.1, Q304.2 (C), Q306.1 (D), R319.1, TR301.6
- net T_POS: now also TR301.7; no longer TR301.8
- net T_NEG: now reaches D311.1 (K), Q303.3 (S), Q305.2 (C), R320.2
- net T_NEG: now also TR301.10, TR301.9; no longer TR301.5, TR301.7
- net at TR301.3: no longer D306.2 (A)
- new net: D306.2 (A), TR301.5
- new net RTN: NT301.2, U301.9 (RTN)
Changed lines of the file:
@@
 $EndDescr
 Wire Wire Line
-	10000 1300 10100 1300
-Wire Wire Line
-	10100 1300 10100 1600
-Wire Wire Line
-	10100 1600 10000 1600
-Wire Wire Line
-	10000 1800 10200 1800
-Wire Wire Line
-	10200 1800 10200 1500
-Wire Wire Line
-	10200 1500 10000 1500
-Connection ~ 10100 1300
-Wire Wire Line
-	10200 1500 10400 1500
-Connection ~ 10200 1500
-Wire Wire Line
-	9600 1800 9500 1800
-Wire Wire Line
-	9500 1800 9500 1900
+	9600 1600 9500 1600
+Wire Wire Line
+	9500 1600 9500 1900
 $Comp
 L unlockoslo:GND_ETH #PWR0123
@@
 Connection ~ 15250 1300
 Wire Wire Line
-	10100 1300 10700 1300
-Wire Wire Line
 	10400 2900 11000 2900
 Wire Wire Line
@@
 Wire Wire Line
 	4900 7800 5000 7800
-Wire Wire Line
-	5000 7800 5000 7700
 Connection ~ 4800 7600
 Wire Wire Line
@@
 Wire Wire Line
 	3950 7600 4800 7600
-Connection ~ 5000 7700
-Wire Wire Line
-	5000 7700 5000 7300
 Wire Wire Line
 	7700 7000 7700 7100
@@
 Text Label 6050 5700 2    50   ~ 0
 CS
-Connection ~ 4800 7700
-Wire Wire Line
-	4800 7700 5000 7700
 Wire Wire Line
 	4800 7300 4800 7600
@@
 Wire Wire Line
 	7500 7500 9250 7500
-Wire Wire Line
-	9250 1600 9600 1600
 $Comp
 L unlockoslo:GND_ETH #PWR0153
@@
 $EndComp
 Wire Wire Line
-	3800 4000 3800 4200
-Wire Wire Line
 	3800 3700 3800 3500
 Wire Wire Line
@@
 Wire Wire Line
 	8500 1500 9600 1500
-Wire Wire Line
-	9250 1600 9250 7500
 Wire Wire Line
 	3650 6400 3300 6400
@@
 	7000 5700 7000 5600
 $Comp
-L Transformer:TRANSF6 TR301
+L unlockoslo:PA2649NL TR301
 U 1 1 5CD663EC
 P 9800 1600
@@
 F 0 "R319" H 11670 1741 50  0000 L CNN
 F 1 "2k" H 11670 1650 50  0000 L CNN
-F 2 "IPC-7351-RESC:RESC_1005x015" V 11530 1650 50  0001 C CNN
+F 2 "IPC-7351-RESC:RESC_3216x040" V 11530 1650 50  0001 C CNN
 F 3 "~" H 11600 1650 50  0001 C CNN
 F 4 "0.25W" H 11670 1559 50  0000 L CNN "Power"
@@
 	1    3650 6150
 	1    0    0    -1
-$EndComp
-$Comp
-L Device:Net-Tie_3_Tee NT301
-U 1 1 5CD23D95
-P 4800 7800
-F 0 "NT301" H 4800 7889 50  0000 C CNN
-F 1 "Net-Tie_3_Tee" H 4800 7980 50  0001 C CNN
-F 2 "NetTie:NetTie-4_SMD_Pad0.5mm" H 4800 7800 50  0001 C CNN
-F 3 "~" H 4800 7800 50  0001 C CNN
-	1    4800 7800
-	-1   0    0    1
 $EndComp
 $Comp
@@
 F 0 "R311" H 6870 6041 50  0000 L CNN
 F 1 "120m" H 6870 5950 50  0000 L CNN
-F 2 "IPC-7351-RESC:RESC_1005x015" V 6730 5950 50  0001 C CNN
+F 2 "IPC-7351-RESC:RESC_3216x040" V 6730 5950 50  0001 C CNN
 F 3 "~" H 6800 5950 50  0001 C CNN
-F 4 "12W" H 6870 5859 50  0000 L CNN "power"
+F 4 "0.25W" H 6870 5859 50  0000 L CNN "power"
+F 5 "RL1206FR-070R12L" H 6800 5950 50  0001 C CNN "mpn"
 	1    6800 5950
 	1    0    0    -1
@@
 $EndComp
 NoConn ~ 5500 5900
+Text Label 10300 1300 2    50   ~ 0
+T_POS
+Text Label 10300 1500 2    50   ~ 0
+T_NEG
+Wire Notes Line
+	7500 10150 7500 8000
+Wire Notes Line width 10
+	7500 8000 9800 8000
+Wire Notes Line
+	9800 8000 9800 600
+Text Label 5500 6900 0    50   ~ 0
+CTL
+Text Label 5500 7000 0    50   ~ 0
+VB
+Wire Wire Line
+	10000 1300 10700 1300
+Wire Wire Line
+	10000 1500 10400 1500
+Wire Wire Line
+	9600 1800 9250 1800
+Wire Wire Line
+	9250 1800 9250 7500
+Text Label 4800 7300 3    50   ~ 0
+ARTN
+Wire Wire Line
+	5000 7300 5000 7800
+Text Label 5000 7500 1    50   ~ 0
+RTN
+Connection ~ 2950 6600
+$Comp
+L power:PWR_FLAG #FLG0101
+U 1 1 5D3AB696
+P 2950 6500
+F 0 "#FLG0101" H 2950 6575 50  0001 C CNN
+F 1 "PWR_FLAG" H 2950 6673 50  0001 C CNN
+F 2 "" H 2950 6500 50  0001 C CNN
+F 3 "~" H 2950 6500 50  0001 C CNN
+	1    2950 6500
+	1    0    0    -1
+$EndComp
+Wire Wire Line
+	2950 6500 2950 6600
+$Comp
+L power:PWR_FLAG #FLG0108
+U 1 1 5D3DEB19
+P 3700 4100
+F 0 "#FLG0108" H 3700 4175 50  0001 C CNN
+F 1 "PWR_FLAG" H 3700 4273 50  0001 C CNN
+F 2 "" H 3700 4100 50  0001 C CNN
+F 3 "~" H 3700 4100 50  0001 C CNN
+	1    3700 4100
+	1    0    0    -1
+$EndComp
+Wire Wire Line
+	3700 4100 3800 4100
+Wire Wire Line
+	3800 4000 3800 4100
+Wire Wire Line
+	3800 4100 3800 4200
+Connection ~ 3800 4100
+$Comp
+L Device:Net-Tie_3_Tee NT301
+U 1 1 5CD23D95
+P 4800 7800
+F 0 "NT301" H 4800 7889 50  0000 C CNN
+F 1 "Net-Tie_3_Tee" H 4800 7980 50  0001 C CNN
+F 2 "NetTie:NetTie-3_SMD_Pad0.5mm" H 4800 7800 50  0001 C CNN
+F 3 "~" H 4800 7800 50  0001 C CNN
+	1    4800 7800
+	1    0    0    1
+$EndComp
+$Comp
+L unlockoslo:GND_ETH #PWR0184
+U 1 1 5D44A100
+P 5700 1900
+F 0 "#PWR0184" H 5700 1650 50  0001 C CNN
+F 1 "GND_ETH" H 5705 1727 50  0000 C CNN
+F 2 "" H 5700 1900 50  0001 C CNN
+F 3 "" H 5700 1900 50  0001 C CNN
+	1    5700 1900
+	1    0    0    -1
+$EndComp
+Wire Wire Line
+	5700 1900 5700 1800
+Connection ~ 5700 1800
+Text Label 5750 6600 0    50   ~ 0
+GAT2
 $EndSCHEMATC

Commit message: o Adjusting a couple of symbols. o PoE done for now.
Parts:
- Q303: symbol Device:Q_NMOS_DGS -> unlockoslo:Q_NMOS_SSSGD
- Q306: symbol Device:Q_NMOS_DGS -> unlockoslo:Q_NMOS_SSSGDDDD
Connections:
- net GND: now also Q303.5 (D), Q306.1 (S), Q306.2 (S); no longer Q303.1 (D)
- net T_NEG: now also Q303.1 (S), Q303.2 (S)
- net T_POS: now also Q306.5 (D), Q306.6 (D), Q306.7 (D), Q306.8 (D); no longer Q306.1 (D)
- net at D311.2 (A), Q305.3 (E): now also Q306.4 (G); no longer Q306.2 (G)
- net at D309.2 (A), Q304.3 (E): now also Q303.4 (G); no longer Q303.2 (G)
Changed lines of the file:
@@
 	10400 1500 10400 2400
 Wire Wire Line
-	14000 2200 14000 2900
-Wire Wire Line
-	14000 1800 14000 1300
+	14000 2200 14000 2300
+Wire Wire Line
+	14000 1800 14000 1700
 Connection ~ 14000 1300
 Wire Wire Line
@@
 Connection ~ 15250 1300
 Wire Wire Line
-	10400 2900 11000 2900
+	10400 2900 10900 2900
 Wire Wire Line
 	14000 2900 13300 2900
@@
 	11600 2800 11600 2900
 Connection ~ 11600 2900
-Wire Wire Line
-	11600 2900 11400 2900
 Wire Wire Line
 	11600 2500 11600 1900
@@
 $EndComp
 $Comp
-L Device:Q_NMOS_DGS Q306
+L unlockoslo:Q_NMOS_SSSGDDDD Q306
 U 1 1 5CD3035C
 P 13900 2000
@@
 	1    15250 2050
 	1    0    0    -1
-$EndComp
-$Comp
-L Device:Q_NMOS_DGS Q303
-U 1 1 5CD30E7C
-P 11200 2800
-F 0 "Q303" V 11451 2800 50  0000 C CNN
-F 1 "Si7852DP" V 11542 2800 50  0000 C CNN
-F 2 "Package_SO:PowerPAK_SO-8_Single" H 11400 2900 50  0001 C CNN
-F 3 "http://www.vishay.com/docs/71627/si7852dp.pdf" H 11200 2800 50  0001 C CNN
-F 4 "SI7852DP-T1-E3" H 11200 2800 50  0001 C CNN "mpn"
-	1    11200 2800
-	0    1    1    0
 $EndComp
 $Comp
@@
 Text Label 5750 6600 0    50   ~ 0
 GAT2
+Wire Wire Line
+	11000 3000 10900 3000
+Wire Wire Line
+	10900 3000 10900 2900
+Connection ~ 10900 2900
+Wire Wire Line
+	10900 2900 11000 2900
+Wire Wire Line
+	11000 3100 10900 3100
+Wire Wire Line
+	10900 3100 10900 3000
+Connection ~ 10900 3000
+Wire Wire Line
+	11400 2900 11600 2900
+$Comp
+L unlockoslo:Q_NMOS_SSSGD Q303
+U 1 1 5CD30E7C
+P 11200 2800
+F 0 "Q303" V 11000 2500 50  0000 C CNN
+F 1 "Si7852DP" V 11750 2800 50  0000 C CNN
+F 2 "Package_SO:PowerPAK_SO-8_Single" H 11400 2900 50  0001 C CNN
+F 3 "http://www.vishay.com/docs/71627/si7852dp.pdf" H 11200 2800 50  0001 C CNN
+F 4 "SI7852DP-T1-E3" H 11200 2800 50  0001 C CNN "mpn"
+	1    11200 2800
+	0    1    1    0
+$EndComp
+Wire Wire Line
+	14100 2200 14100 2300
+Wire Wire Line
+	14100 2300 14000 2300
+Connection ~ 14000 2300
+Wire Wire Line
+	14000 2300 14000 2900
+Wire Wire Line
+	14100 2300 14200 2300
+Wire Wire Line
+	14200 2300 14200 2200
+Connection ~ 14100 2300
+Wire Wire Line
+	14100 1800 14100 1700
+Wire Wire Line
+	14100 1700 14000 1700
+Connection ~ 14000 1700
+Wire Wire Line
+	14000 1700 14000 1300
+Wire Wire Line
+	14100 1700 14200 1700
+Wire Wire Line
+	14200 1700 14200 1800
+Connection ~ 14100 1700
+Wire Wire Line
+	14200 1700 14300 1700
+Wire Wire Line
+	14300 1700 14300 1800
+Connection ~ 14200 1700
 $EndSCHEMATC
