File: pcb/base-1.0/power-mux.sch (KiCad schematic (older format))
At the start: 23 parts

Commit message: wip
Parts:
- gave numbers to parts that had none: 23
Changed lines of the file:
@@
 $EndDescr
 $Comp
-L Device:Q_PMOS_DGS Q?
+L Device:Q_PMOS_DGS Q201
 U 1 1 5CF241D9
 P 4900 1800
-F 0 "Q?" V 5243 1800 50  0000 C CNN
+F 0 "Q201" V 5243 1800 50  0000 C CNN
 F 1 "Q_PMOS_DGS" V 5152 1800 50  0000 C CNN
 F 2 "" H 5100 1900 50  0001 C CNN
@@
 Connection ~ 5200 2200
 $Comp
-L Device:C C?
+L Device:C C204
 U 1 1 5CF2798D
 P 4900 2450
-F 0 "C?" H 5015 2496 50  0000 L CNN
+F 0 "C204" H 5015 2496 50  0000 L CNN
 F 1 "100n" H 5015 2405 50  0000 L CNN
 F 2 "" H 4938 2300 50  0001 C CNN
@@
 	4900 2200 4900 2300
 $Comp
-L power:GND #PWR?
+L power:GND #PWR0112
 U 1 1 5CF2B26C
 P 4900 2700
-F 0 "#PWR?" H 4900 2450 50  0001 C CNN
+F 0 "#PWR0112" H 4900 2450 50  0001 C CNN
 F 1 "GND" H 4905 2527 50  0000 C CNN
 F 2 "" H 4900 2700 50  0001 C CNN
@@
 	4900 2700 4900 2600
 $Comp
-L Device:Q_PMOS_DGS Q?
+L Device:Q_PMOS_DGS Q203
 U 1 1 5CF4269A
 P 6700 2000
-F 0 "Q?" V 7043 2000 50  0000 C CNN
+F 0 "Q203" V 7043 2000 50  0000 C CNN
 F 1 "Q_PMOS_DGS" V 6952 2000 50  0000 C CNN
 F 2 "" H 6900 2100 50  0001 C CNN
@@
 $EndComp
 $Comp
-L Device:Q_PMOS_DGS Q?
+L Device:Q_PMOS_DGS Q204
 U 1 1 5CF426A0
 P 7300 2000
-F 0 "Q?" V 7643 2000 50  0000 C CNN
+F 0 "Q204" V 7643 2000 50  0000 C CNN
 F 1 "Q_PMOS_DGS" V 7552 2000 50  0000 C CNN
 F 2 "" H 7500 2100 50  0001 C CNN
@@
 Connection ~ 7000 2400
 $Comp
-L Device:C C?
+L Device:C C205
 U 1 1 5CF426B0
 P 6700 2650
-F 0 "C?" H 6815 2696 50  0000 L CNN
+F 0 "C205" H 6815 2696 50  0000 L CNN
 F 1 "100n" H 6815 2605 50  0000 L CNN
 F 2 "" H 6738 2500 50  0001 C CNN
@@
 	6700 2400 6700 2500
 $Comp
-L power:GND #PWR?
+L power:GND #PWR0113
 U 1 1 5CF426B7
 P 6700 2900
-F 0 "#PWR?" H 6700 2650 50  0001 C CNN
+F 0 "#PWR0113" H 6700 2650 50  0001 C CNN
 F 1 "GND" H 6705 2727 50  0000 C CNN
 F 2 "" H 6700 2900 50  0001 C CNN
@@
 	6700 2900 6700 2800
 $Comp
-L Device:Q_PMOS_DGS Q?
+L Device:Q_PMOS_DGS Q205
 U 1 1 5CF45010
 P 8500 2200
-F 0 "Q?" V 8843 2200 50  0000 C CNN
+F 0 "Q205" V 8843 2200 50  0000 C CNN
 F 1 "Q_PMOS_DGS" V 8752 2200 50  0000 C CNN
 F 2 "" H 8700 2300 50  0001 C CNN
@@
 $EndComp
 $Comp
-L Device:Q_PMOS_DGS Q?
+L Device:Q_PMOS_DGS Q206
 U 1 1 5CF45016
 P 9100 2200
-F 0 "Q?" V 9443 2200 50  0000 C CNN
+F 0 "Q206" V 9443 2200 50  0000 C CNN
 F 1 "Q_PMOS_DGS" V 9352 2200 50  0000 C CNN
 F 2 "" H 9300 2300 50  0001 C CNN
@@
 Connection ~ 8800 2600
 $Comp
-L Device:C C?
+L Device:C C206
 U 1 1 5CF45026
 P 8500 2850
-F 0 "C?" H 8615 2896 50  0000 L CNN
+F 0 "C206" H 8615 2896 50  0000 L CNN
 F 1 "100n" H 8615 2805 50  0000 L CNN
 F 2 "" H 8538 2700 50  0001 C CNN
@@
 	8500 2600 8500 2700
 $Comp
-L power:GND #PWR?
+L power:GND #PWR0114
 U 1 1 5CF4502D
 P 8500 3100
-F 0 "#PWR?" H 8500 2850 50  0001 C CNN
+F 0 "#PWR0114" H 8500 2850 50  0001 C CNN
 F 1 "GND" H 8505 2927 50  0000 C CNN
 F 2 "" H 8500 3100 50  0001 C CNN
@@
 	8100 800  8100 2100
 $Comp
-L Device:R R?
+L Device:R R201
 U 1 1 5CF7BBFC
 P 1400 2450
-F 0 "R?" H 1470 2496 50  0000 L CNN
+F 0 "R201" H 1470 2496 50  0000 L CNN
 F 1 "R" H 1470 2405 50  0000 L CNN
 F 2 "" V 1330 2450 50  0001 C CNN
@@
 $EndComp
 $Comp
-L Device:R R?
+L Device:R R202
 U 1 1 5CF7BE8C
 P 1400 2950
-F 0 "R?" H 1470 2996 50  0000 L CNN
+F 0 "R202" H 1470 2996 50  0000 L CNN
 F 1 "R" H 1470 2905 50  0000 L CNN
 F 2 "" V 1330 2950 50  0001 C CNN
@@
 $EndComp
 $Comp
-L Device:R R?
+L Device:R R203
 U 1 1 5CF7C8AE
 P 1400 3450
-F 0 "R?" H 1470 3496 50  0000 L CNN
+F 0 "R203" H 1470 3496 50  0000 L CNN
 F 1 "49,9k" H 1470 3405 50  0000 L CNN
 F 2 "" V 1330 3450 50  0001 C CNN
@@
 	1400 3100 1400 3200
 $Comp
-L power:GND #PWR?
+L power:GND #PWR0115
 U 1 1 5CF7FE7C
 P 1400 3700
-F 0 "#PWR?" H 1400 3450 50  0001 C CNN
+F 0 "#PWR0115" H 1400 3450 50  0001 C CNN
 F 1 "GND" H 1405 3527 50  0000 C CNN
 F 2 "" H 1400 3700 50  0001 C CNN
@@
 	1400 2700 1400 2800
 $Comp
-L Device:R R?
+L Device:R R204
 U 1 1 5CF88E5C
 P 2100 2450
-F 0 "R?" H 2170 2496 50  0000 L CNN
+F 0 "R204" H 2170 2496 50  0000 L CNN
 F 1 "R" H 2170 2405 50  0000 L CNN
 F 2 "" V 2030 2450 50  0001 C CNN
@@
 $EndComp
 $Comp
-L Device:R R?
+L Device:R R205
 U 1 1 5CF88E66
 P 2100 2950
-F 0 "R?" H 2170 2996 50  0000 L CNN
+F 0 "R205" H 2170 2996 50  0000 L CNN
 F 1 "R" H 2170 2905 50  0000 L CNN
 F 2 "" V 2030 2950 50  0001 C CNN
@@
 $EndComp
 $Comp
-L Device:R R?
+L Device:R R206
 U 1 1 5CF88E70
 P 2100 3450
-F 0 "R?" H 2170 3496 50  0000 L CNN
+F 0 "R206" H 2170 3496 50  0000 L CNN
 F 1 "R" H 2170 3405 50  0000 L CNN
 F 2 "" V 2030 3450 50  0001 C CNN
@@
 	2100 3100 2100 3200
 $Comp
-L power:GND #PWR?
+L power:GND #PWR0116
 U 1 1 5CF88E7C
 P 2100 3700
-F 0 "#PWR?" H 2100 3450 50  0001 C CNN
+F 0 "#PWR0116" H 2100 3450 50  0001 C CNN
 F 1 "GND" H 2105 3527 50  0000 C CNN
 F 2 "" H 2100 3700 50  0001 C CNN
@@
 	2100 2700 2100 2800
 $Comp
-L Device:R R?
+L Device:R R207
 U 1 1 5CF99158
 P 2800 2450
-F 0 "R?" H 2870 2496 50  0000 L CNN
+F 0 "R207" H 2870 2496 50  0000 L CNN
 F 1 "R" H 2870 2405 50  0000 L CNN
 F 2 "" V 2730 2450 50  0001 C CNN
@@
 $EndComp
 $Comp
-L Device:R R?
+L Device:R R208
 U 1 1 5CF99162
 P 2800 2950
-F 0 "R?" H 2870 2996 50  0000 L CNN
+F 0 "R208" H 2870 2996 50  0000 L CNN
 F 1 "R" H 2870 2905 50  0000 L CNN
 F 2 "" V 2730 2950 50  0001 C CNN
@@
 $EndComp
 $Comp
-L Device:R R?
+L Device:R R209
 U 1 1 5CF9916C
 P 2800 3450
-F 0 "R?" H 2870 3496 50  0000 L CNN
+F 0 "R209" H 2870 3496 50  0000 L CNN
 F 1 "R" H 2870 3405 50  0000 L CNN
 F 2 "" V 2730 3450 50  0001 C CNN
@@
 $EndComp
 $Comp
-L power:GND #PWR?
+L power:GND #PWR0117
 U 1 1 5CF99178
 P 2800 3700
-F 0 "#PWR?" H 2800 3450 50  0001 C CNN
+F 0 "#PWR0117" H 2800 3450 50  0001 C CNN
 F 1 "GND" H 2805 3527 50  0000 C CNN
 F 2 "" H 2800 3700 50  0001 C CNN
@@
 	10200 5500 10200 3400
 $Comp
-L unlockoslo:Net-Tie_3_to_1 NT?
+L unlockoslo:Net-Tie_3_to_1 NT201
 U 1 1 5D02029B
 P 10000 3400
-F 0 "NT?" H 10000 3581 50  0000 C CNN
+F 0 "NT201" H 10000 3581 50  0000 C CNN
 F 1 "Net-Tie_4_to_1" H 10000 3490 50  0000 C CNN
 F 2 "" H 10000 3400 50  0001 C CNN
@@
 	10200 3400 10650 3400
 $Comp
-L power:GND #PWR?
+L power:GND #PWR0118
 U 1 1 5D02AAC7
 P 4500 7300
-F 0 "#PWR?" H 4500 7050 50  0001 C CNN
+F 0 "#PWR0118" H 4500 7050 50  0001 C CNN
 F 1 "GND" H 4505 7127 50  0000 C CNN
 F 2 "" H 4500 7300 50  0001 C CNN
@@
 	4500 7300 4500 7200
 $Comp
-L LTC4417:LTC4417 U?
+L LTC4417:LTC4417 U201
 U 1 1 5D0392DB
 P 4500 6100
-F 0 "U?" H 4500 6100 50  0000 C CNN
+F 0 "U201" H 4500 6100 50  0000 C CNN
 F 1 "LTC4417" H 4500 6000 50  0000 C CNN
 F 2 "" H 4500 6400 50  0001 C CNN
@@
 Vin_USB
 $Comp
-L Device:C C?
+L Device:C C203
 U 1 1 5D042E21
 P 3000 1600
-F 0 "C?" H 3115 1646 50  0000 L CNN
+F 0 "C203" H 3115 1646 50  0000 L CNN
 F 1 "100n" H 3115 1555 50  0000 L CNN
 F 2 "" H 3038 1450 50  0001 C CNN
@@
 $EndComp
 $Comp
-L Device:C C?
+L Device:C C201
 U 1 1 5D04EC39
 P 1600 1600
-F 0 "C?" H 1715 1646 50  0000 L CNN
+F 0 "C201" H 1715 1646 50  0000 L CNN
 F 1 "100n" H 1715 1555 50  0000 L CNN
 F 2 "" H 1638 1450 50  0001 C CNN
@@
 $EndComp
 $Comp
-L Device:C C?
+L Device:C C202
 U 1 1 5D0490E5
 P 2300 1600
-F 0 "C?" H 2415 1646 50  0000 L CNN
+F 0 "C202" H 2415 1646 50  0000 L CNN
 F 1 "100n" H 2415 1555 50  0000 L CNN
 F 2 "" H 2338 1450 50  0001 C CNN
@@
 	1600 1450 1600 1350
 $Comp
-L power:GND #PWR?
+L power:GND #PWR0119
 U 1 1 5D066DDE
 P 1600 1850
-F 0 "#PWR?" H 1600 1600 50  0001 C CNN
+F 0 "#PWR0119" H 1600 1600 50  0001 C CNN
 F 1 "GND" H 1605 1677 50  0000 C CNN
 F 2 "" H 1600 1850 50  0001 C CNN
@@
 $EndComp
 $Comp
-L power:GND #PWR?
+L power:GND #PWR0120
 U 1 1 5D06712D
 P 2300 1850
-F 0 "#PWR?" H 2300 1600 50  0001 C CNN
+F 0 "#PWR0120" H 2300 1600 50  0001 C CNN
 F 1 "GND" H 2305 1677 50  0000 C CNN
 F 2 "" H 2300 1850 50  0001 C CNN
@@
 $EndComp
 $Comp
-L power:GND #PWR?
+L power:GND #PWR0121
 U 1 1 5D067423
 P 3000 1850
-F 0 "#PWR?" H 3000 1600 50  0001 C CNN
+F 0 "#PWR0121" H 3000 1600 50  0001 C CNN
 F 1 "GND" H 3005 1677 50  0000 C CNN
 F 2 "" H 3000 1850 50  0001 C CNN
@@
 NoConn ~ 5600 6700
 $Comp
-L power:GND #PWR?
+L power:GND #PWR0122
 U 1 1 5D1CDC51
 P 5700 6900
-F 0 "#PWR?" H 5700 6650 50  0001 C CNN
+F 0 "#PWR0122" H 5700 6650 50  0001 C CNN
 F 1 "GND" H 5705 6727 50  0000 C CNN
 F 2 "" H 5700 6900 50  0001 C CNN
@@
 	5700 6800 5700 6900
 $Comp
-L Device:Q_PMOS_DGS Q?
+L Device:Q_PMOS_DGS Q202
 U 1 1 5CF24862
 P 5500 1800
-F 0 "Q?" V 5843 1800 50  0000 C CNN
+F 0 "Q202" V 5843 1800 50  0000 C CNN
 F 1 "Q_PMOS_DGS" V 5752 1800 50  0000 C CNN
 F 2 "" H 5700 1900 50  0001 C CNN

Commit message: wip
Connections:
- net ~Valid1 renamed ~Valid_PoE
- net ~Valid2 renamed ~Valid_adapter
- net ~Valid3 renamed ~Valid_USB
Changed lines of the file:
@@
 $Descr A4 11693 8268
 encoding utf-8
-Sheet 4 3
+Sheet 2 3
 Title ""
 Date ""
@@
 	6200 6200 5600 6200
 Text HLabel 6200 6000 2    50   Input ~ 0
-~Valid1
+~Valid_PoE
 Text HLabel 6200 6100 2    50   Input ~ 0
-~Valid2
+~Valid_adapter
 Text HLabel 6200 6200 2    50   Input ~ 0
-~Valid3
+~Valid_USB
 NoConn ~ 5600 6500
 NoConn ~ 5600 6600

Commit message: wip
Parts:
- C201, C202, C203, C204, C205, C206: footprint (none) -> Capacitor_SMD:C_0402_1005Metric
- NT201: footprint (none) -> NetTie:NetTie-4_SMD_Pad0.5mm
- R201, R202, R203, R204, R205, R206, R207, R208, R209: footprint (none) -> Resistor_SMD:R_0402_1005Metric
Changed lines of the file:
@@
 F 0 "C204" H 5015 2496 50  0000 L CNN
 F 1 "100n" H 5015 2405 50  0000 L CNN
-F 2 "" H 4938 2300 50  0001 C CNN
+F 2 "Capacitor_SMD:C_0402_1005Metric" H 4938 2300 50  0001 C CNN
 F 3 "~" H 4900 2450 50  0001 C CNN
 	1    4900 2450
@@
 F 0 "C205" H 6815 2696 50  0000 L CNN
 F 1 "100n" H 6815 2605 50  0000 L CNN
-F 2 "" H 6738 2500 50  0001 C CNN
+F 2 "Capacitor_SMD:C_0402_1005Metric" H 6738 2500 50  0001 C CNN
 F 3 "~" H 6700 2650 50  0001 C CNN
 	1    6700 2650
@@
 F 0 "C206" H 8615 2896 50  0000 L CNN
 F 1 "100n" H 8615 2805 50  0000 L CNN
-F 2 "" H 8538 2700 50  0001 C CNN
+F 2 "Capacitor_SMD:C_0402_1005Metric" H 8538 2700 50  0001 C CNN
 F 3 "~" H 8500 2850 50  0001 C CNN
 	1    8500 2850
@@
 F 0 "R201" H 1470 2496 50  0000 L CNN
 F 1 "R" H 1470 2405 50  0000 L CNN
-F 2 "" V 1330 2450 50  0001 C CNN
+F 2 "Resistor_SMD:R_0402_1005Metric" V 1330 2450 50  0001 C CNN
 F 3 "~" H 1400 2450 50  0001 C CNN
 	1    1400 2450
@@
 F 0 "R202" H 1470 2996 50  0000 L CNN
 F 1 "R" H 1470 2905 50  0000 L CNN
-F 2 "" V 1330 2950 50  0001 C CNN
+F 2 "Resistor_SMD:R_0402_1005Metric" V 1330 2950 50  0001 C CNN
 F 3 "~" H 1400 2950 50  0001 C CNN
 	1    1400 2950
@@
 F 0 "R203" H 1470 3496 50  0000 L CNN
 F 1 "49,9k" H 1470 3405 50  0000 L CNN
-F 2 "" V 1330 3450 50  0001 C CNN
+F 2 "Resistor_SMD:R_0402_1005Metric" V 1330 3450 50  0001 C CNN
 F 3 "~" H 1400 3450 50  0001 C CNN
 	1    1400 3450
@@
 F 0 "R204" H 2170 2496 50  0000 L CNN
 F 1 "R" H 2170 2405 50  0000 L CNN
-F 2 "" V 2030 2450 50  0001 C CNN
+F 2 "Resistor_SMD:R_0402_1005Metric" V 2030 2450 50  0001 C CNN
 F 3 "~" H 2100 2450 50  0001 C CNN
 	1    2100 2450
@@
 F 0 "R205" H 2170 2996 50  0000 L CNN
 F 1 "R" H 2170 2905 50  0000 L CNN
-F 2 "" V 2030 2950 50  0001 C CNN
+F 2 "Resistor_SMD:R_0402_1005Metric" V 2030 2950 50  0001 C CNN
 F 3 "~" H 2100 2950 50  0001 C CNN
 	1    2100 2950
@@
 F 0 "R206" H 2170 3496 50  0000 L CNN
 F 1 "R" H 2170 3405 50  0000 L CNN
-F 2 "" V 2030 3450 50  0001 C CNN
+F 2 "Resistor_SMD:R_0402_1005Metric" V 2030 3450 50  0001 C CNN
 F 3 "~" H 2100 3450 50  0001 C CNN
 	1    2100 3450
@@
 F 0 "R207" H 2870 2496 50  0000 L CNN
 F 1 "R" H 2870 2405 50  0000 L CNN
-F 2 "" V 2730 2450 50  0001 C CNN
+F 2 "Resistor_SMD:R_0402_1005Metric" V 2730 2450 50  0001 C CNN
 F 3 "~" H 2800 2450 50  0001 C CNN
 	1    2800 2450
@@
 F 0 "R208" H 2870 2996 50  0000 L CNN
 F 1 "R" H 2870 2905 50  0000 L CNN
-F 2 "" V 2730 2950 50  0001 C CNN
+F 2 "Resistor_SMD:R_0402_1005Metric" V 2730 2950 50  0001 C CNN
 F 3 "~" H 2800 2950 50  0001 C CNN
 	1    2800 2950
@@
 F 0 "R209" H 2870 3496 50  0000 L CNN
 F 1 "R" H 2870 3405 50  0000 L CNN
-F 2 "" V 2730 3450 50  0001 C CNN
+F 2 "Resistor_SMD:R_0402_1005Metric" V 2730 3450 50  0001 C CNN
 F 3 "~" H 2800 3450 50  0001 C CNN
 	1    2800 3450
@@
 F 0 "NT201" H 10000 3581 50  0000 C CNN
 F 1 "Net-Tie_4_to_1" H 10000 3490 50  0000 C CNN
-F 2 "" H 10000 3400 50  0001 C CNN
+F 2 "NetTie:NetTie-4_SMD_Pad0.5mm" H 10000 3400 50  0001 C CNN
 F 3 "~" H 10000 3400 50  0001 C CNN
 	1    10000 3400
@@
 F 0 "C203" H 3115 1646 50  0000 L CNN
 F 1 "100n" H 3115 1555 50  0000 L CNN
-F 2 "" H 3038 1450 50  0001 C CNN
+F 2 "Capacitor_SMD:C_0402_1005Metric" H 3038 1450 50  0001 C CNN
 F 3 "~" H 3000 1600 50  0001 C CNN
 	1    3000 1600
@@
 F 0 "C201" H 1715 1646 50  0000 L CNN
 F 1 "100n" H 1715 1555 50  0000 L CNN
-F 2 "" H 1638 1450 50  0001 C CNN
+F 2 "Capacitor_SMD:C_0402_1005Metric" H 1638 1450 50  0001 C CNN
 F 3 "~" H 1600 1600 50  0001 C CNN
 	1    1600 1600
@@
 F 0 "C202" H 2415 1646 50  0000 L CNN
 F 1 "100n" H 2415 1555 50  0000 L CNN
-F 2 "" H 2338 1450 50  0001 C CNN
+F 2 "Capacitor_SMD:C_0402_1005Metric" H 2338 1450 50  0001 C CNN
 F 3 "~" H 2300 1600 50  0001 C CNN
 	1    2300 1600

Commit message: wip
Parts:
- added R210, R211, R212: 1M, Resistor_SMD:R_0402_1005Metric, symbol Device:R
Connections:
- net Vout: now also R210.1, R211.1, R212.1
- net ~Valid_PoE: now also R210.2
- net ~Valid_USB: now also R212.2
- net ~Valid_adapter: now also R211.2
Changed lines of the file:
@@
 F 1 "LTC4417" H 4500 6000 50  0000 C CNN
 F 2 "" H 4500 6400 50  0001 C CNN
-F 3 "" H 4500 6400 50  0001 C CNN
+F 3 "http://www.linear.com/docs/42408" H 4500 6400 50  0001 C CNN
 	1    4500 6100
 	1    0    0    -1
@@
 	1400 800  8100 800
 Wire Wire Line
-	5600 5500 10200 5500
-Wire Wire Line
-	5600 6000 6200 6000
-Wire Wire Line
-	6200 6100 5600 6100
-Wire Wire Line
-	6200 6200 5600 6200
-Text HLabel 6200 6000 2    50   Input ~ 0
+	5600 5500 5700 5500
+Wire Wire Line
+	5600 6000 5700 6000
+Wire Wire Line
+	6650 6100 6100 6100
+Wire Wire Line
+	6650 6200 6500 6200
+Text HLabel 6650 6000 2    50   Input ~ 0
 ~Valid_PoE
-Text HLabel 6200 6100 2    50   Input ~ 0
+Text HLabel 6650 6100 2    50   Input ~ 0
 ~Valid_adapter
-Text HLabel 6200 6200 2    50   Input ~ 0
+Text HLabel 6650 6200 2    50   Input ~ 0
 ~Valid_USB
 NoConn ~ 5600 6500
@@
 Text Notes 2400 -850 0    50   ~ 0
 TODO:\n* Select MOSFETs. One option: CSD75207W15\n* Calculate resistor values
+$Comp
+L Device:R R210
+U 1 1 5D207874
+P 5700 5750
+F 0 "R210" H 5770 5796 50  0000 L CNN
+F 1 "1M" H 5770 5705 50  0000 L CNN
+F 2 "Resistor_SMD:R_0402_1005Metric" V 5630 5750 50  0001 C CNN
+F 3 "~" H 5700 5750 50  0001 C CNN
+	1    5700 5750
+	1    0    0    -1
+$EndComp
+$Comp
+L Device:R R211
+U 1 1 5D207BF4
+P 6100 5750
+F 0 "R211" H 6170 5796 50  0000 L CNN
+F 1 "1M" H 6170 5705 50  0000 L CNN
+F 2 "Resistor_SMD:R_0402_1005Metric" V 6030 5750 50  0001 C CNN
+F 3 "~" H 6100 5750 50  0001 C CNN
+	1    6100 5750
+	1    0    0    -1
+$EndComp
+$Comp
+L Device:R R212
+U 1 1 5D207E7A
+P 6500 5750
+F 0 "R212" H 6570 5796 50  0000 L CNN
+F 1 "1M" H 6570 5705 50  0000 L CNN
+F 2 "Resistor_SMD:R_0402_1005Metric" V 6430 5750 50  0001 C CNN
+F 3 "~" H 6500 5750 50  0001 C CNN
+	1    6500 5750
+	1    0    0    -1
+$EndComp
+Wire Wire Line
+	6500 5900 6500 6200
+Connection ~ 6500 6200
+Wire Wire Line
+	6500 6200 5600 6200
+Wire Wire Line
+	6100 5900 6100 6100
+Connection ~ 6100 6100
+Wire Wire Line
+	6100 6100 5600 6100
+Wire Wire Line
+	5700 5900 5700 6000
+Connection ~ 5700 6000
+Wire Wire Line
+	5700 6000 6650 6000
+Wire Wire Line
+	5700 5600 5700 5500
+Connection ~ 5700 5500
+Wire Wire Line
+	5700 5500 6100 5500
+Wire Wire Line
+	6100 5600 6100 5500
+Connection ~ 6100 5500
+Wire Wire Line
+	6100 5500 6500 5500
+Wire Wire Line
+	6500 5600 6500 5500
+Connection ~ 6500 5500
+Wire Wire Line
+	6500 5500 10200 5500
 $EndSCHEMATC

Commit message: wip
Parts:
- U201: footprint (none) -> Package_DFN_QFN:QFN-24-1EP_4x4mm_P0.5mm_EP2.6x2.6mm_ThermalVias
Connections:
- net GND: now also U201.25 (EP)
Changed lines of the file:
@@
 L power:GND #PWR0118
 U 1 1 5D02AAC7
-P 4500 7300
-F 0 "#PWR0118" H 4500 7050 50  0001 C CNN
-F 1 "GND" H 4505 7127 50  0000 C CNN
-F 2 "" H 4500 7300 50  0001 C CNN
-F 3 "" H 4500 7300 50  0001 C CNN
-	1    4500 7300
-	1    0    0    -1
-$EndComp
-Wire Wire Line
-	4500 7300 4500 7200
+P 4500 7400
+F 0 "#PWR0118" H 4500 7150 50  0001 C CNN
+F 1 "GND" H 4505 7227 50  0000 C CNN
+F 2 "" H 4500 7400 50  0001 C CNN
+F 3 "" H 4500 7400 50  0001 C CNN
+	1    4500 7400
+	1    0    0    -1
+$EndComp
+Wire Wire Line
+	4500 7400 4500 7300
 $Comp
 L LTC4417:LTC4417 U201
@@
 F 0 "U201" H 4500 6100 50  0000 C CNN
 F 1 "LTC4417" H 4500 6000 50  0000 C CNN
-F 2 "" H 4500 6400 50  0001 C CNN
+F 2 "Package_DFN_QFN:QFN-24-1EP_4x4mm_P0.5mm_EP2.6x2.6mm_ThermalVias" H 4500 6400 50  0001 C CNN
 F 3 "http://www.linear.com/docs/42408" H 4500 6400 50  0001 C CNN
 	1    4500 6100
@@
 Wire Wire Line
 	6500 5500 10200 5500
+Wire Wire Line
+	4600 7200 4600 7300
+Wire Wire Line
+	4600 7300 4500 7300
+Connection ~ 4500 7300
+Wire Wire Line
+	4500 7300 4500 7200
 $EndSCHEMATC
