File: pcb/base-1.0/power-mux.sch (KiCad schematic (older format))
At the start: 24 parts, among them Q201 IRF7324TRPBF, Q202 IRF7324TRPBF, Q203 IRF7324TRPBF, U201 LTC4417

Commit message: o More MPNs. o Ignoring DPN parts from BOM. o Changing from TL431D to TL431DBV, has a smaller footprint.
Parts:
- U201: mpn (none) -> LTC4417CUF#TRPBF
Changed lines of the file:
@@
 F 2 "Package_DFN_QFN:QFN-24-1EP_4x4mm_P0.5mm_EP2.6x2.6mm_ThermalVias" H 4500 6400 50  0001 C CNN
 F 3 "http://www.linear.com/docs/42408" H 4500 6400 50  0001 C CNN
+F 4 "LTC4417CUF#TRPBF" H 4500 6100 50  0001 C CNN "mpn"
 	1    4500 6100
 	1    0    0    -1
