File: pcb/base-1.0/base-1.0.sch (KiCad schematic (older format))
At the start: 50 parts, among them J101 USB_B_Micro, J102 Conn_01x06, J103 74984104400, J104 Jack-DC, Q101 BC817, Q102 BC817, Q103 DMP2305U-7, SW101 SW_Push, U101 CP2102N-A01-GQFN24, U102 LAN8720A, U103 ESP32-WROOM-32D, U104 USBLC6-2SC6

Commit message: wip
Parts:
- C113, C114: footprint Capacitors_SMD:C_0402 -> Capacitor_SMD:C_0402_1005Metric
- FB102: footprint Inductors_SMD:L_0402 -> Inductor_SMD:L_0402_1005Metric
- J101: footprint (none) -> 10118194:10118194; mpn (none) -> 10118194-0001LF
- Q103: footprint TO_SOT_Packages_SMD:SOT-23 -> Package_TO_SOT_SMD:SOT-23
Changed lines of the file:
@@
 F 0 "J101" H 857 2167 50  0000 C CNN
 F 1 "USB_B_Micro" H 857 2076 50  0000 C CNN
-F 2 "" H 950 1650 50  0001 C CNN
-F 3 "~" H 950 1650 50  0001 C CNN
+F 2 "10118194:10118194" H 950 1650 50  0001 C CNN
+F 3 "https://www.amphenol-icc.com/media/wysiwyg/files/drawing/10118194.pdf" H 950 1650 50  0001 C CNN
+F 4 "10118194-0001LF" H 800 1700 50  0001 C CNN "mpn"
 	1    800  1700
 	1    0    0    -1
@@
 F 0 "Q103" V 4743 6600 50  0000 C CNN
 F 1 "DMP2305U-7" V 4652 6600 50  0000 C CNN
-F 2 "TO_SOT_Packages_SMD:SOT-23" H 4600 6700 50  0001 C CNN
+F 2 "Package_TO_SOT_SMD:SOT-23" H 4600 6700 50  0001 C CNN
 F 3 "~" H 4400 6600 50  0001 C CNN
 	1    4400 6600
@@
 F 0 "FB102" V 1263 1200 50  0000 C CNN
 F 1 "MPZ1005S900HT000" V 1354 1200 50  0000 C CNN
-F 2 "Inductors_SMD:L_0402" V 1430 1200 50  0001 C CNN
+F 2 "Inductor_SMD:L_0402_1005Metric" V 1430 1200 50  0001 C CNN
 F 3 "~" H 1500 1200 50  0001 C CNN
 	1    1500 1200
@@
 F 0 "C113" H 815 2441 50  0000 L CNN
 F 1 "C" H 815 2350 50  0000 L CNN
-F 2 "Capacitors_SMD:C_0402" H 738 2200 50  0001 C CNN
+F 2 "Capacitor_SMD:C_0402_1005Metric" H 738 2200 50  0001 C CNN
 F 3 "~" H 700 2350 50  0001 C CNN
 F 4 "DNP" H 815 2259 50  0000 L CNN "populate"
@@
 F 0 "C114" H 9315 1796 50  0000 L CNN
 F 1 "1u" H 9315 1705 50  0000 L CNN
-F 2 "Capacitors_SMD:C_0402" H 9238 1600 50  0001 C CNN
+F 2 "Capacitor_SMD:C_0402_1005Metric" H 9238 1600 50  0001 C CNN
 F 3 "~" H 9200 1750 50  0001 C CNN
 	1    9200 1750

Commit message: wip
Parts:
- J102: footprint (none) -> Connector_PinHeader_2.54mm:PinHeader_1x06_P2.54mm_Vertical
Other:
- note added: "TODO:\n* Ethernet PHY\n * LED polarities\n* Ethernet PoE\n* ORing\n * Add valid LEDs. Note that they're biased against Vout.\n* Cuttable PCB traces for LEDs to enable low power?\n* Test points:\n * Power in\n * Important data signals\n* Connectors\n * UEXT (x2?)\n* Check footprints of all parts\n * footprint\n * pins"
- note removed: "TODO:\n* Ethernet PHY\n * LED polarities\n* Ethernet PoE\n* ORing\n * Add valid LEDs. Note that they're biased against Vout.\n* Cuttable PCB traces for LEDs to enable low power?\n* Test points:\n * Power in\n * Important data signals\n* Connectors\n * UEXT (x2?)\n* Check footprints of all parts"
Changed lines of the file:
@@
 TODO:\no use QFN20 part\no Move TXT/RXT
 Text Notes 150  -50  0    50   ~ 0
-TODO:\n* Ethernet PHY\n  * LED polarities\n* Ethernet PoE\n* ORing\n  * Add valid LEDs. Note that they're biased against Vout.\n* Cuttable PCB traces for LEDs to enable low power?\n* Test points:\n  * Power in\n  * Important data signals\n* Connectors\n  * UEXT (x2?)\n* Check footprints of all parts
+TODO:\n* Ethernet PHY\n  * LED polarities\n* Ethernet PoE\n* ORing\n  * Add valid LEDs. Note that they're biased against Vout.\n* Cuttable PCB traces for LEDs to enable low power?\n* Test points:\n  * Power in\n  * Important data signals\n* Connectors\n  * UEXT (x2?)\n* Check footprints of all parts\n  * footprint\n  * pins
 $Comp
 L Device:R R104
@@
 F 0 "J102" V 5814 412 50  0000 R CNN
 F 1 "Conn_01x06" V 5723 412 50  0000 R CNN
-F 2 "" H 5850 800 50  0001 C CNN
+F 2 "Connector_PinHeader_2.54mm:PinHeader_1x06_P2.54mm_Vertical" H 5850 800 50  0001 C CNN
 F 3 "~" H 5850 800 50  0001 C CNN
 	1    5850 800

Commit message: wip
Parts:
- added C103: 4.7uF, symbol Device:C
- added C115: 100nF, symbol Device:C
- added J105: USB_GPIO, symbol Connector_Generic:Conn_01x02
- D103: value LED -> RX
- D104: value LED -> TX
- J102: value Conn_01x06 -> UART; symbol Connector_Generic:Conn_01x06 -> unlockoslo:Conn_UART_5
Connections:
- net labels added: +3.3V_USB
- wire segments 256 -> 271
- no-connect marks 15 -> 19
Other:
- note added: "Debugging UART only.\nCan not power the device."
- note added: "Should RTS/DTR be swapped too?"
- note removed: "TODO:\no Decoupling?"
- note removed: "TODO:\no use QFN20 part\no Move TXT/RXT"
- moved on the sheet: C113, C114, D103, D104, FB102, J101, Q101, Q102, R101, R102, R104, R106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

Commit message: wip
Parts:
- C103, C115: footprint (none) -> Capacitor_SMD:C_0402_1005Metric
- J105: footprint (none) -> Connector_PinHeader_2.54mm:PinHeader_1x02_P2.54mm_Vertical
Changed lines of the file:
@@
 F 0 "C115" H 3815 1496 50  0000 L CNN
 F 1 "100nF" H 3815 1405 50  0000 L CNN
-F 2 "" H 3738 1300 50  0001 C CNN
+F 2 "Capacitor_SMD:C_0402_1005Metric" H 3738 1300 50  0001 C CNN
 F 3 "~" H 3700 1450 50  0001 C CNN
 	1    3700 1450
@@
 F 0 "C103" H 3286 1404 50  0000 R CNN
 F 1 "4.7uF" H 3286 1495 50  0000 R CNN
-F 2 "" H 3438 1300 50  0001 C CNN
+F 2 "Capacitor_SMD:C_0402_1005Metric" H 3438 1300 50  0001 C CNN
 F 3 "~" H 3400 1450 50  0001 C CNN
 	1    3400 1450
@@
 F 0 "J105" H 7030 2392 50  0000 L CNN
 F 1 "USB_GPIO" H 7030 2301 50  0000 L CNN
-F 2 "" H 6950 2400 50  0001 C CNN
+F 2 "Connector_PinHeader_2.54mm:PinHeader_1x02_P2.54mm_Vertical" H 6950 2400 50  0001 C CNN
 F 3 "~" H 6950 2400 50  0001 C CNN
 	1    6950 2400
@@
 Should RTS/DTR be swapped too?
 $Comp
-L unlockoslo:+3.3V_USB #PWR?
+L unlockoslo:+3.3V_USB #PWR0109
 U 1 1 5D64632A
 P 6500 2800
-F 0 "#PWR?" H 6500 2650 50  0001 C CNN
+F 0 "#PWR0109" H 6500 2650 50  0001 C CNN
 F 1 "+3.3V_USB" H 6515 2973 50  0000 C CNN
 F 2 "" H 6500 2800 50  0001 C CNN

Commit message: wip
Parts:
- added C? (x4): 0.1u, IPC7351-Nominal:CAPC2012X70, symbol Device:C
- added C? (x4): 22u, IPC7351-Nominal:CAPC2012X70, symbol Device:C
- added C? (x2): 75p, IPC7351-Nominal:CAPC1005X55, symbol Device:C
- added C? (x2): 10u, IPC7351-Nominal:CAPC2012X70, symbol Device:C
- added D? (x2): POWER, IPC7351-Nominal:LEDC3216X110, symbol Device:LED
- added J?: Raspberry_Pi_2_3, symbol Connector:Raspberry_Pi_2_3
- added L? (x2): 15u, Inductors_SMD:L_Taiyo-Yuden_NR-80xx, symbol Device:L_Core_Ferrite
- added P? (x2): 12V, Bitraf:har-flexicon_2,54_TSPH-02_T56_BK, symbol Connector_Generic:Conn_01x02
- added R? (x2): 560, IPC7351-Nominal:RESC1005X38, symbol Device:R
- added R? (x2): 100k, IPC7351-Nominal:RESC1005X38, symbol Device:R
- added R? (x2): 13.3k, IPC7351-Nominal:RESC1005X38, symbol Device:R
- added TP? (x2): +5V, Connectors_TestPoints:Test_Point_Pad_d1.0mm, symbol Connector:TestPoint
- added U? (x2): TPS54202, TO_SOT_Packages_SMD:SOT-23-6_Handsoldering, symbol tps54202:TPS54202
Connections:
- net +3V3: now also R116.2; no longer R116.1
- net ETH_GREEN_P: now also R116.1; no longer R116.2
- net GND: now also C?.2, C?.2, C?.2, C?.2, C?.2, C?.2, C?.2, C?.2, J?.14 (GND), J?.20 (GND), J?.25 (GND), J?.30 (GND), J?.34 (GND), J?.39 (GND), J?.6 (GND), J?.9 (GND), P?.2 (Pin_2), P?.2 (Pin_2), R?.2, R?.2, R?.2, R?.2, U?.1 (GND), U?.1 (GND)
- net PoE/Vin_A1: no longer J103.7 (V1+)
- net PoE/Vin_A2: no longer J103.8 (V1-)
- net PoE/Vin_B1: no longer J103.9 (V2+)
- net PoE/Vin_B2: no longer J103.10 (V2-)
- net Power mux/Vin_USB: no longer C103.2, C115.1, FB102.1, R101.1, U101.7 (REGIN), U104.5 (VBUS)
- net Power mux/Vin_adapter: no longer J104.1
- new net: C103.2, C115.1, FB102.1, R101.1, U101.7 (REGIN), U104.5 (VBUS)
- new net: D?.1 (K), R?.1 (x2)
- new net +5V: C?.1, C?.1, C?.1, C?.1, C?.1, C?.1, D?.2 (A), D?.2 (A), L?.1, L?.1, R?.1, R?.1, TP?.1, TP?.1
- new net BOOT: C?.1, C?.1, U?.6 (BOOT), U?.6 (BOOT)
- new net FB: C?.2, C?.2, R?.1, R?.1, R?.2, R?.2, U?.4 (FB), U?.4 (FB)
- new net SW: C?.2, C?.2, L?.2, L?.2, U?.2 (SW), U?.2 (SW)
- new net Vin: C?.1, C?.1, C?.1, C?.1, P?.1 (Pin_1), P?.1 (Pin_1), U?.3 (Vin), U?.3 (Vin)
- no-connect marks 19 -> 21
Other:
- note added: "8V - 24 V to 5 V switched mode DC/DC regulator"
- note added: "Capacitors are\nrated to 10V"
- note added: "Capacitors are\nrated to 35V"
- note added: "Design is based on "8.2 Typical Application" from the data sheet.\nThe design supports 8-28 V inputs.\nEN has internal pull up."
- note added: "TODO:\n * LED polarities\n* ORing\n * Add valid LEDs. Note that they're biased against Vout.\n* Adjust DC/DC for 12 V.\n* Test points:\n * Power in\n * Important data signals\n* Connectors\n * UEXT (x2?)\n* Check footprints of all parts\n * footprint\n * pins"
- note removed: "Should RTS/DTR be swapped too?"
- note removed: "TODO:\n* Ethernet PHY\n * LED polarities\n* Ethernet PoE\n* ORing\n * Add valid LEDs. Note that they're biased against Vout.\n* Cuttable PCB traces for LEDs to enable low power?\n* Test points:\n * Power in\n * Important data signals\n* Connectors\n * UEXT (x2?)\n* Check footprints of all parts\n * footprint\n * pins"
- moved on the sheet: C101, C102, C104, C105, C106, C107, C108, C109, C110, C111, C112, C114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

Commit message: wip
Parts:
- removed P? (x2): 12V, Bitraf:har-flexicon_2,54_TSPH-02_T56_BK, symbol Connector_Generic:Conn_01x02
- J106: renamed from J?; footprint (none) -> Connector_PinHeader_2.54mm:PinHeader_2x20_P2.54mm_Vertical
- gave numbers to parts that had none: 26
Connections:
- net PHY_MDC: no longer R110.1, U102.10 (RXER/PHYAD0)
- net PoE/Vin_A1: now also J103.7 (V1+)
- net PoE/Vin_A2: now also J103.8 (V1-)
- net PoE/Vin_B1: now also J103.9 (V2+)
- net PoE/Vin_B2: now also J103.10 (V2-)
- net Power mux/Vin_USB: now also C103.2, C115.1, FB102.1, R101.1, U101.7 (REGIN), U104.5 (VBUS)
- net Power mux/Vin_adapter: now also J104.1
- net +5V: no longer names the net of C122.1, C124.1, C126.1, D101.2 (A), L101.1, R103.1, TP102.1
- net +5V: no longer C123.1, C125.1, C127.1, D102.2 (A), L102.1, R111.1, TP103.1
- new net: R110.1, U102.10 (RXER/PHYAD0)
- new net: C123.1, C125.1, C127.1, D102.2 (A), L102.1, R111.1, TP103.1
Other:
- note added: "TODO:\n * LED polarities\n* ORing\n * Add valid LEDs. Note that they're biased against Vout.\n* Adjust DC/DC for 12 V.\n* Test points:\n * Power in\n * Important data signals\n* Connectors\n * UEXT (x2?)\n* Check footprints of all parts\n * footprint\n * pins\n* Move to IPC footprint library.\n"
- note removed: "8V - 24 V to 5 V switched mode DC/DC regulator"
- note removed: "TODO:\n * LED polarities\n* ORing\n * Add valid LEDs. Note that they're biased against Vout.\n* Adjust DC/DC for 12 V.\n* Test points:\n * Power in\n * Important data signals\n* Connectors\n * UEXT (x2?)\n* Check footprints of all parts\n * footprint\n * pins"
- moved on the sheet: C101, C102, C104, C105, C106, C107, C108, C109, C110, C111, C112, C114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

Commit message: o Replacing footprints with IPC footprints.
Parts:
- C101, C102, C103, C104, C105, C106, C107, C108, C109, C110, C111, C112, C113, C114, C115: footprint Capacitor_SMD:C_0402_1005Metric -> IPC-7351-CAPC:CAPC_1005x015
- C116, C117, C118, C119, C120, C121, C124, C125, C126, C127: footprint IPC7351-Nominal:CAPC2012X70 -> IPC-7351-CAPC:CAPC_2012x040
- C122, C123: footprint IPC7351-Nominal:CAPC1005X55 -> IPC-7351-CAPC:CAPC_1005x015
- D101, D102: footprint IPC7351-Nominal:LEDC3216X110 -> IPC-7351-LEDSC:LEDSC_3216x060
- D103, D104: footprint LED_SMD:LED_1206_3216Metric -> IPC-7351-LEDSC:LEDSC_3216x060
- R101, R102, R104, R106, R107, R108, R109, R110, R112, R113, R114, R115, R116, R117, R118, R119, R120: footprint Resistor_SMD:R_0402_1005Metric -> IPC-7351-RESC:RESC_1005x015
- R103, R105, R111, R121, R122, R123: footprint IPC7351-Nominal:RESC1005X38 -> IPC-7351-RESC:RESC_1005x015

Commit message: o Better symbol for BC817, Q101 and Q102. o Adding footprint for jack, J104.
Parts:
- J104: footprint (none) -> Connector_BarrelJack:BarrelJack_CUI_PJ-063AH_Horizontal; mpn (none) -> PJ-037AH-SMT-TR
- Q101, Q102: symbol Transistor_BJT:BC817 -> Device:Q_NPN_BEC
Changed lines of the file:
@@
 F 0 "J104" H 1057 4725 50  0000 C CNN
 F 1 "Jack-DC" H 1057 4634 50  0000 C CNN
-F 2 "" H 1050 4360 50  0001 C CNN
-F 3 "~" H 1050 4360 50  0001 C CNN
+F 2 "Connector_BarrelJack:BarrelJack_CUI_PJ-063AH_Horizontal" H 1050 4360 50  0001 C CNN
+F 3 "https://www.cui.com/product/resource/pj-037ah-smt-tr.pdf" H 1050 4360 50  0001 C CNN
+F 4 "PJ-037AH-SMT-TR" H 1000 4400 50  0001 C CNN "mpn"
 	1    1000 4400
 	1    0    0    -1
@@
 	5600 2700 7300 2700
 $Comp
-L Transistor_BJT:BC817 Q102
+L Device:Q_NPN_BEC Q102
 U 1 1 5D35866F
 P 9000 2300
@@
 F 1 "BC817" H 9191 2345 50  0000 L CNN
 F 2 "Package_TO_SOT_SMD:SOT-23" H 9200 2225 50  0001 L CIN
-F 3 "http://www.fairchildsemi.com/ds/BC/BC817.pdf" H 9000 2300 50  0001 L CNN
+F 3 "https://assets.nexperia.com/documents/data-sheet/BC817_SER.pdf" H 9000 2300 50  0001 L CNN
 	1    9000 2300
 	1    0    0    1
 $EndComp
 $Comp
-L Transistor_BJT:BC817 Q101
+L Device:Q_NPN_BEC Q101
 U 1 1 5D3585A1
 P 9000 1600
@@
 F 1 "BC817" H 9191 1555 50  0000 L CNN
 F 2 "Package_TO_SOT_SMD:SOT-23" H 9200 1525 50  0001 L CIN
-F 3 "http://www.fairchildsemi.com/ds/BC/BC817.pdf" H 9000 1600 50  0001 L CNN
+F 3 "https://assets.nexperia.com/documents/data-sheet/BC817_SER.pdf" H 9000 1600 50  0001 L CNN
 	1    9000 1600
 	1    0    0    -1
