File: pcb/base-1.0/base-1.0.sch (KiCad schematic (older format))
At the start: 86 parts, among them J101 USB_B_Micro, J102 UART, J103 74984104400, J104 Jack-DC, J105 USB_GPIO, J106 RPI_HEADER, Q101 BC817, Q102 BC817, Q103 DMP2305U-7, SW101 TL3315NF100Q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

Commit message: o More PCB work.
Parts:
- removed C109: 1uF, IPC-7351-CAPC:CAPC_1005x015, symbol Device:C
- removed RN101: 49.9 Ω, Resistor_SMD:R_Array_Convex_4x1206, symbol Device:R_Pack04
- added R124, R125, R126, R127: 49.9, IPC-7351-RESC:RESC_1005x015, symbol Device:R
Connections:
- net PoE/Vin_B2 is gone; now on net PoE/Vin_A1: J103.10 (V2-)
- net +3V3: now also C108.1
- net +3V3_PHY: now also R124.1, R125.1, R126.1, R127.1; no longer C108.1, R116.2
- net D+: now also U104.6 (IO1); no longer U104.4 (IO2)
- net D-: now also U104.4 (IO2); no longer U104.3 (IO2)
- net ETH_GREEN_N: now also U102.3 (LED1/REGOFF); no longer U102.2 (LED2/nINTSEL)
- net ETH_RD+: now also R126.2
- net ETH_RD-: now also R127.2
- net ETH_TD+: now also R124.2
- net ETH_TD-: now also R125.2
- net ETH_YELLOW_P: now also U102.2 (LED2/nINTSEL); no longer U102.3 (LED1/REGOFF)
- net EXP_A0: now also J106.37 (GPIO26); no longer J106.27 (ID_SD/GPIO0)
- net EXP_A1: now also J106.36 (GPIO16); no longer J106.28 (ID_SC/GPIO1)
- net EXP_A2: now also J106.31 (GCLK2/GPIO6); no longer J106.7 (GCLK0/GPIO4)
- net EXP_A4: now also J106.28 (ID_SC/GPIO1); no longer J106.31 (GCLK2/GPIO6)
- net EXP_A5: now also J106.27 (ID_SD/GPIO0); no longer J106.26 (~CE1~/GPIO7)
- net EXP_A6: now also J106.26 (~CE1~/GPIO7); no longer J106.24 (~CE0~/GPIO8)
- net EXP_A7: now also J106.24 (~CE0~/GPIO8); no longer J106.21 (MISO0/GPIO9)
- net EXP_B0: now also J106.22 (GPIO25); no longer J106.36 (GPIO16)
- net EXP_B1: now also J106.21 (MISO0/GPIO9); no longer J106.11 (GPIO17)
- net EXP_B2: now also J106.18 (GPIO24); no longer J106.15 (GPIO22)
- net EXP_B4: now also J106.15 (GPIO22); no longer J106.18 (GPIO24)
- net EXP_B5: now also J106.13 (GPIO27); no longer J106.22 (GPIO25)
- net EXP_B6: now also J106.11 (GPIO17); no longer J106.37 (GPIO26)
- net EXP_B7: now also J106.7 (GCLK0/GPIO4); no longer J106.13 (GPIO27)
- net PHY_VDDA: now also R116.2
- net Power mux/Vin_USB: no longer U104.5 (VBUS)
- net at FB102.2, J101.1 (VBUS): now also U104.5 (VBUS)
- net IN_D-: now reaches J101.2 (D-)
- net IN_D-: now also U104.3 (IO2); no longer U104.6 (IO1)
- net IN_D+: now reaches J101.3 (D+), U104.1 (IO1)
Other:
- note added: "VDDCR: output from LAN8720 internal 1.2V regulator.\nLED 1: link activity, green\nLED 2: Link speed, yellow"
- note removed: "VDDCR is output from LAN8720 internal 1.2V regulator."
- moved on the sheet: C104, C107, C108, C113, FB102, J101, J103, R108, R115, R116, U104

Commit message: o More PCB work.
Parts:
- NT101, NT102: footprint NetTie:NetTie-2_SMD_Pad0.5mm -> UnlockOslo:NetTie-2_SMD_Pad0.15mm
Changed lines of the file:
@@
 F 0 "NT101" H 6400 1889 50  0001 C CNN
 F 1 "Net-Tie_2" H 6400 1890 50  0001 C CNN
-F 2 "NetTie:NetTie-2_SMD_Pad0.5mm" H 6400 1800 50  0001 C CNN
+F 2 "UnlockOslo:NetTie-2_SMD_Pad0.15mm" H 6400 1800 50  0001 C CNN
 F 3 "~" H 6400 1800 50  0001 C CNN
 	1    6400 1800
@@
 F 0 "NT102" H 6400 1811 50  0001 C CNN
 F 1 "Net-Tie_2" H 6400 1990 50  0001 C CNN
-F 2 "NetTie:NetTie-2_SMD_Pad0.5mm" H 6400 1900 50  0001 C CNN
+F 2 "UnlockOslo:NetTie-2_SMD_Pad0.15mm" H 6400 1900 50  0001 C CNN
 F 3 "~" H 6400 1900 50  0001 C CNN
 	1    6400 1900
