File: pcb/base-1.0/base-1.0.kicad_pcb (KiCad board)
At the start: 2 copper layers, 85.6 x 54 mm, 182 parts, among them J101 USB_B_Micro, J102 UART, J103 74984104400, J104 Jack-DC, J105 USB_GPIO, J106 RPI_HEADER, Q101 BC817, Q102 BC817, Q103 DMP2305U-7, Q201 IRF7324TRPBF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

Commit message: o 4 layers.
Parts:
- removed NT301, NT302: Net-Tie_3, UnlockOslo:NetTie-3_SMD_Pad0.5mm_132
- added NT201: Net-Tie_3_to_1, NetTie:NetTie-4_SMD_Pad0.5mm, F.Cu at (149.6, 97.7)
- NT203: footprint UnlockOslo:NetTie-2_SMD_Pad0.15mm -> UnlockOslo:NetTie-2_SMD_Pad0.20mm
- moved TP102 50.7 mm to (47.5, 1.60)
- moved R210 26.1 mm to (155.8, 87.8), turned to 0 degrees
- moved R211 25.6 mm to (155.8, 86.8), turned to 0 degrees
- moved R212 25.2 mm to (155.8, 85.8), turned to 0 degrees
- moved Q203 23.1 mm to (161.5, 99.2), turned to 0 degrees
- moved C206 21.7 mm to (157.0, 98.0)
- moved R208 7.04 mm to (132.1, 97.8)
- moved U201 5.52 mm to (138.7, 93.9), turned to 90 degrees
- moved R207 5.29 mm to (131.1, 97.8), turned to 90 degrees
- moved R209 4.92 mm to (133.1, 97.8), turned to 270 degrees
- moved C203 3.80 mm to (127.8, 94.4)
- moved C128 2.64 mm to (133.0, 88.3)
- moved NT202 1.58 mm to (151.9, 112.2)
- moved NT203 0.60 mm to (140.2, 116.5)
- moved NT102 0.07 mm to (121.9, 95.1)
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Connections:
- net /PoE/ETH_VDD renamed /PoE/VDD_ETH
- net /PoE/ETH_VSS renamed /PoE/VSS_ETH
- net /Power mux/OV1 renamed Net-(R208-Pad2)
- net /Power mux/OV2 renamed Net-(R205-Pad2)
- net /Power mux/OV3 renamed Net-(R202-Pad2)
- net /Power mux/UV1 renamed Net-(R207-Pad2)
- net /Power mux/UV2 renamed Net-(R204-Pad2)
- net /Power mux/UV3 renamed Net-(R201-Pad2)
Routing:
- net /PHY_VDDA: track 12.6 -> 59.2 mm, vias 2 -> 4
- net /EXP_A0: track 23.7 -> 0.00 mm
- net Net-(Q202-Pad2): track 26.7 -> 4.17 mm, vias 2 -> 0
- net /EXP_A1: track 22.3 -> 0.00 mm
- net GND: track 96.2 -> 115.3 mm, vias 31 -> 28
- net Net-(NT301-Pad2): track 18.6 -> 0.00 mm
- net Net-(Q201-Pad2): track 21.5 -> 4.19 mm, vias 2 -> 0
- net GND_ETH: track 31.8 -> 48.3 mm, vias 17 -> 31
- net /EXP_A2: track 15.5 -> 0.00 mm
- net /DTR: track 18.2 -> 2.88 mm, vias 1 -> 0
- net /ETH_YELLOW_P: track 56.6 -> 41.7 mm
- net Net-(C204-Pad1): track 21.9 -> 7.13 mm, vias 2 -> 0
- net /EXP_A4: track 14.3 -> 0.00 mm
- net Net-(C205-Pad1): track 21.0 -> 7.05 mm, vias 2 -> 0
- net /Power mux/Vin_adapter: track 29.2 -> 16.4 mm, vias 2 -> 0
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- added copper zone on In2.Cu, net +3V3
- added copper zone on F.Cu, net /PoE/VDD_ETH
- added copper zone on B.Cu, net /PoE/VSS_ETH
- added copper zone on In1.Cu, net GND
- added copper zone on In1.Cu, net GND_ETH
- removed copper zone on B.Cu, net GND_ETH
Other:
- copper layers 2 -> 4
- net class Size_0.10__0.5 removed

Commit message: o More PCB work.
Parts:
- removed NT201: Net-Tie_3_to_1, NetTie:NetTie-4_SMD_Pad0.5mm
- added NT1: Net-Tie_3, UnlockOslo:NetTie-3_SMD_Pad0.5mm_132, F.Cu at (146.0, 90.3)
- added NT2: Net-Tie_3, UnlockOslo:NetTie-3_SMD_Pad0.5mm_132, F.Cu at (130.8, 91.8)
- L303: footprint 744770122:744770122 -> Inductor_SMD:L_Taiyo-Yuden_NR-80xx
- moved U103 32.5 mm to (245.1, 90.5)
- moved C202 16.7 mm to (138.2, 99.0), turned to 180 degrees
- moved R204 16.1 mm to (141.2, 99.0), turned to 0 degrees
- moved R206 15.3 mm to (138.2, 98.0), turned to 180 degrees
- moved R205 14.7 mm to (141.2, 98.0), turned to 180 degrees
- moved R210 14.6 mm to (142.8, 94.3), turned to 180 degrees
- moved R211 14.6 mm to (142.8, 93.3), turned to 180 degrees
- moved R212 14.6 mm to (142.8, 92.3), turned to 180 degrees
- moved C206 9.28 mm to (149.2, 93.0)
- moved Q203 9.28 mm to (153.7, 94.2)
- moved C201 9.00 mm to (144.5, 87.6)
- moved R201 9.00 mm to (145.5, 87.6)
- moved R202 9.00 mm to (146.5, 87.6)
- moved R203 9.00 mm to (147.5, 87.6)
- moved Q306 4.79 mm to (186.2, 113.4), turned to 180 degrees
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Connections:
- D302 pad 4: /PoE/Vin_A1 -> /PoE/Vin_B2
- J103 pad 10: /PoE/Vin_A1 -> /PoE/Vin_B2
Routing:
- net /PoE/T_POS: track 0.00 -> 30.0 mm
- net /DTR: track 2.88 -> 30.6 mm, vias 0 -> 1
- net /Power mux/Vin_USB: track 65.7 -> 40.3 mm, vias 8 -> 6
- net /EXP_A0: track 0.00 -> 23.7 mm
- net /EXP_A1: track 0.00 -> 22.6 mm
- net Net-(C205-Pad1): track 7.05 -> 29.0 mm, vias 0 -> 2
- net Net-(D311-Pad2): track 0.00 -> 21.7 mm
- net GND: track 115.3 -> 136.7 mm, vias 28 -> 44
- net /RTS: track 9.90 -> 30.6 mm
- net Net-(C204-Pad1): track 7.13 -> 27.0 mm, vias 0 -> 2
- net Net-(Q202-Pad2): track 4.17 -> 23.9 mm, vias 0 -> 2
- net Net-(Q201-Pad2): track 4.19 -> 22.4 mm, vias 0 -> 2
- net /EXP_A2: track 0.00 -> 15.5 mm
- net /MCU_IO32: track 0.00 -> 15.4 mm, vias 0 -> 1
- net /EXP_A4: track 0.00 -> 14.7 mm
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