File: pcb/base-1.0/base-1.0.kicad_pcb (KiCad board)
At the start: 4 copper layers, 85.6 x 54 mm, 182 parts, among them J101 USB_B_Micro, J102 UART, J103 74984104400, J104 Jack-DC, J105 USB_GPIO, J106 RPI_HEADER, Q101 BC817, Q102 BC817, Q103 DMP2305U-7, Q201 IRF7324TRPBF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

Commit message: o More PCB work.
Parts:
- added H105: MountingHole, MountingHole:MountingHole_2.5mm, F.Cu at (81.0, 128.0)
- added H106: MountingHole, MountingHole:MountingHole_2.5mm, F.Cu at (81.0, 80.0)
- NT203: moved to B.Cu
- R320: footprint IPC-7351-RESC:RESC_1005x015 -> IPC-7351-RESC:RESC_3216x040
- moved C120 125.5 mm to (140.8, 44.0)
- moved C122 125.5 mm to (144.7, 44.9)
- moved D101 125.5 mm to (159.8, 52.3)
- moved L101 125.5 mm to (154.2, 46.0)
- moved R103 125.5 mm to (144.7, 43.9)
- moved R105 125.5 mm to (144.7, 42.9)
- moved R122 125.5 mm to (158.2, 51.3)
- moved TP102 125.5 mm to (163.2, 50.4)
- moved U105 125.5 mm to (145.1, 47.2)
- moved C116 125.5 mm to (149.9, 44.5)
- moved C118 125.5 mm to (147.9, 44.5)
- moved C124 125.5 mm to (151.9, 50.5)
- moved C126 125.5 mm to (151.9, 52.5)
- moved C117 93.9 mm to (112.0, 46.2)
- moved C119 93.9 mm to (112.0, 48.2)
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Routing:
- net /ETH_GREEN_P: track 2.23 -> 66.2 mm
- net Net-(C104-Pad1): track 0.00 -> 58.5 mm
- net /PHY_VDDA: track 59.2 -> 1.22 mm, vias 4 -> 0
- net /ETH_YELLOW_N: track 2.36 -> 52.9 mm
- net /PoE/VDD_ETH: track 44.5 -> 8.01 mm
- net /PoE/CTL: track 29.7 -> 0.00 mm, vias 2 -> 0
- net /ETH_RD-: track 34.2 -> 59.8 mm
- net /ETH_RD+: track 33.5 -> 56.3 mm
- net /ETH_GREEN_N: track 47.8 -> 69.0 mm, vias 1 -> 0
- net /ETH_TD+: track 38.0 -> 57.7 mm
- net /PoE/VC: track 18.6 -> 0.00 mm, vias 2 -> 0
- net GND: track 136.7 -> 118.3 mm, vias 44 -> 34
- net /ETH_TD-: track 37.2 -> 55.5 mm
- net /MCU_RX: track 20.1 -> 2.37 mm
- net Net-(D311-Pad2): track 21.7 -> 4.85 mm
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- added copper zone on F.Cu, net /PoE/VSS_ETH
- added copper zone on B.Cu, net GND_ETH
- removed copper zone on B.Cu, net /PoE/VSS_ETH
- removed copper zone on In1.Cu, net GND_ETH
Other:
- board size 85.6 x 54 mm -> 115.6 x 54 mm

Commit message: o More PCB work.
Parts:
- moved R309 19.4 mm to (130.2, 113.5), turned to 270 degrees
- moved C304 18.8 mm to (129.2, 113.5), turned to 270 degrees
- moved R310 17.9 mm to (129.2, 110.5), turned to 270 degrees
- moved C310 17.0 mm to (130.2, 110.5), turned to 270 degrees
- moved D305 16.6 mm to (133.1, 109.8)
- moved D306 16.6 mm to (136.2, 109.8)
- moved L301 11.6 mm to (130.2, 105.8), turned to 90 degrees
- moved C307 11.4 mm to (124.3, 106.8), turned to 180 degrees
- moved C308 10.2 mm to (125.3, 105.3), turned to 180 degrees
- moved C312 3.78 mm to (134.2, 107.0)
- moved D307 3.78 mm to (136.7, 106.9)
- moved Q302 3.78 mm to (139.3, 106.8)
- moved R308 3.78 mm to (133.2, 107.0)
- moved R313 3.78 mm to (135.2, 107.0)
- moved C315 2.96 mm to (142.1, 107.5)
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Routing:
- net /PoE/CTL: track 0.00 -> 18.9 mm, vias 0 -> 2
- net /PoE/GAT2: track 0.00 -> 15.9 mm, vias 0 -> 2
- net /PoE/VC: track 0.00 -> 10.3 mm
- net /PoE/VB: track 0.00 -> 9.95 mm, vias 0 -> 2
- net Net-(D306-Pad2): track 0.00 -> 9.16 mm
- net Net-(D305-Pad1): track 0.00 -> 6.72 mm
- net Net-(C315-Pad2): track 17.7 -> 23.0 mm
- net Net-(C312-Pad1): track 0.00 -> 4.37 mm
- net Net-(C301-Pad1): track 7.54 -> 11.7 mm
- net Net-(Q301-Pad4): track 0.00 -> 3.65 mm
- net /PoE/GATE: track 17.6 -> 21.3 mm
- net Net-(C313-Pad1): track 1.58 -> 5.12 mm
- net /PoE/CS: track 20.1 -> 17.0 mm, vias 3 -> 2
- net Net-(C301-Pad2): track 12.3 -> 15.2 mm
- net Net-(C315-Pad1): track 0.00 -> 1.97 mm
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